File: board/olchanowski.sch (EAGLE design)
At the start: 68 parts, among them IC1 LPC1768, J1 B4B-XH-A(LF)(SN), J2 B4B-XH-A(LF)(SN), J3 B4B-XH-A(LF)(SN), U1 TMC2209-LA, U2 TMC2209-LA, U3 TMC2209-LA, U4 TMC2209-LA

Commit message: Added ethernet
Parts:
- added C47, C48, C49, C50, C51, C52, C53, C54, C55, C56, C57, C58, C59, C60, C61, C62: (no value), rcl:C-EUC0402
- added J4: ARJM11D7-009-AB-ER2-T, robbe:ARJM11D7-009-AB-ER2-T
- added Q2: (no value), crystal:CRYSTALHC49UP
- added R13, R14, R15, R16, R17, R18, R19, R20, R21, R22, R23, R24, R25, R26, R27: (no value), rcl:R-US_R0402
- added U5: LAN8720, microchip-smsc-lan8720:LAN8720
- added U6: 74HC1G04, SparkFun-IC-Logic:74HC1G04
Connections:
- new net ENET_CRS: IC1.P1[8]/ENET_CRS, R21.1
- new net ENET_LED1: J4.LED_L_A, U5.LED1/REGOFF
- new net ENET_LED2: J4.LED_R_A, R26.2, U5.LED2/!INTSEL
- new net ENET_MDC: IC1.P1[16]/ENET_MDC, U5.MDC
- new net ENET_MDIO: IC1.P1[17]/ENET_MDIO, R24.1, U5.MDIO
- new net ENET_REF_CLK: IC1.P1[15]/ENET_REF_CLK, R20.2
- new net ENET_RXD0: IC1.P1[9]/ENET_RXD0, R23.1
- new net ENET_RXD1: IC1.P1[10]/ENET_RXD1, R22.1
- new net ENET_RX_ER: IC1.P1[14]/ENET_RX_ER, R25.1, U5.RXER/PHYAD0
- new net ENET_TXD0: IC1.P1[0]/ENET_TXD0, U5.TXD0
- new net ENET_TXD1: IC1.P1[1]/ENET_TXD1, U5.TXD1
- new net ENET_TXD_EN: IC1.P1[4]/ENET_TX_EN
- new net ENET_TX_EN: U5.TXEN
- new net N$39: C52.1, J4.TD+, R18.2, U5.TXP
- new net N$40: C51.1, J4.TD-, R17.2, U5.TXN
- new net N$41: C50.1, J4.RD+, R16.2, U5.RXP
- new net N$43: C49.1, J4.RD-, R15.2, U5.RXN
- new net N$44: J4.LED_R_C, R13.2
- new net N$45: J4.LED_L_C, R14.2
- new net N$46: U5.REFCLKO/!INT, U6G1.A
- new net N$47: C53.1, Q2.2, R19.2, U5.XTAL2
- new net N$48: C54.1, Q2.1, R19.1, U5.XTAL1/CLKIN
- new net N$49: C55.2, C56.1, U5.VDDCR
- new net N$50: R20.1, U6G1.Y
- new net N$51: R21.2, U5.CRS_DV/MODE2
- new net N$52: R22.2, U5.RXD1/MODE1
- new net N$53: R23.2, U5.RXD0/MODE0
- new net N$54: R27.2, U5.RBIAS
- new net RSTOUT: IC1.RSTOUT, U5.!RST
- net +3V3: now also C47.2, C48.2, C57.2, C58.1, C59.2, C60.2, C61.2, C62.2, J4.RCT, J4.TCT, R15.1, R16.1, R17.1, R18.1, R24.2, R25.2, U5.VDD1A, U5.VDD2A, U5.VDDIO, U6G2.P$V+
- net GND: now also C47.1, C48.1, C49.2, C50.2, C51.2, C52.2, C53.2, C54.2, C55.1, C56.2, C57.1, C58.2, C59.1, C60.1, C61.1, C62.1, J4.GND, J4.SHIELD1, J4.SHIELD2, R13.1, R14.1, R26.1, R27.1, U5.VSS, U6G2.P$V-
Other:
- note added: "ETHERNET"

Commit message: Endstops and heater drivers
Parts:
- added C63, C64: (no value), rcl:C-EUC0402
- added Q3, Q4: SIJA58DP, robbe:SIJA58DP
- added R28, R29, R30, R31, R32: (no value), rcl:R-US_R0402
- added U7: LM5111, robbe:LM5111
- added X1, X2, X3: X-AXIS, JST_XH:JST-XH-02-PIN-LONG-PAD
Connections:
- new net +5V: C63.2, C64.2, U7.VCC
- new net EXTR_HEATER_EN: IC1.P2[7]/RD2/RTS1, R32.2, U7.INB
- new net HB_EN: IC1.P2[5]/PWM1[6]/DTR1/TRACEDATA[0], R31.2, U7.INA
- new net N$55: Q4.G, U7.OUTA
- new net N$56: Q3.G, U7.OUTB
- new net X_END: IC1.P1[24]/MCI2/PWM1[5]/MOSI0, R28.1, X1-2.S
- new net Y_END: IC1.P1[26]/MCOB1/PWM1[6]/CAP0[0], R29.1, X2-2.S
- new net Z_END: IC1.P1[28]/MCOA2/PCAP1[0]/MAT0[0], R30.1, X3-2.S
- net +3V3: now also R28.2, R29.2, R30.2
- net GND: now also C63.1, C64.1, Q3.S, Q4.S, R31.1, R32.1, U7.VEE, X1-1.S, X2-1.S, X3-1.S
Other:
- note added: "END STOPS"
- note added: "HEATER DRIVERS"
- note added: "POWER"
- note added: "TODO: - SMPS: 24V -> 5V - LDO: 5V -> 3V3"
- note added: "TODO: Find connectors"

Commit message: More schematic stuff
Parts:
- added C65, C69, C77: (no value), rcl:CPOL-EU150CLZ-0810
- added C66, C67, C70, C71, C73, C74, C75, C76: 10u, rcl:C-EUC0805
- added C68, C72: (no value), rcl:C-EUC0402
- added J5: B4B-XH-A(LF)(SN), B4B-XH-A_LF__SN_:B4B-XH-A(LF)(SN)
- added P1: TPSM53602, robbe:TPSM53602
- added Q5, Q6, Q7, Q8: SSM3K329R,LF, robbe:SSM3K329R,LF
- added R33, R34, R35, R36, R37, R38, R39, R40: (no value), rcl:R-US_R0402
- added SV1: ICSP, con-lsta:FE06-1
- added SW1, SW2: SPST-2-4PIN, robbe:SPST-2-4PIN
- added U8: NCP5661-0, robbe:NCP5661-0
- added X4: FAN, JST_XH:JST-XH-02-PIN-LONG-PAD
- added X5: UI, con-3m:2520-
Connections:
- new net BTN: X5-9.KL
- new net BUZZER_GATE: X5-3.KL
- new net CTS: SV1.2
- new net FAN_EN: IC1.P2[4]/PWM1[5]/DSR1/TRACEDATA[1], Q5.G, R33.2
- new net LED_B: J5.1, Q6.D
- new net LED_G: J5.3, Q8.D
- new net LED_R: J5.2, Q7.D
- new net N$57: Q5.D, X4-1.S
- new net N$58: P1.FB, R37.2, R38.1
- new net RESET: IC1.RESET, R40.1, SW2.S, SW2.S1
- new net RGB_B: IC1.P1[21]/MCABORT/PWM1[3]/SSEL0, Q6.G, R34.2
- new net RGB_G: IC1.P1[20]/MCI0/PWM1[2]/SCK0, Q8.G, R36.2
- new net RGB_R: IC1.P1[18]/USB_UP_LED/PWM1[1]/CAP1[0], Q7.G, R35.2
- new net ROT_A: X5-11.KL
- new net ROT_B\: X5-12.KL
- new net RTS: SV1.6
- new net RX: IC1.P0[3]/RXD0/AD0[6], SV1.4
- new net SW_ISP: IC1.P2[10]/EINT0/NMI, R39.1, SW1.S, SW1.S1
- new net TX: IC1.P0[2]/TXD0/AD0[7], SV1.5
- net +24V: now also C65.+, C66.1, C67.1, C68.2, J5.4, P1.EN, P1.VIN, X4-2.S
- net +3V3: now also C74.1, C75.1, C77.+, R39.2, R40.2, SV1.3, U8.VOUT, X5-2.KL, X5-20.KL
- net +5V: now also C69.+, C70.1, C71.1, C72.2, C73.1, C76.1, P1.VOUT, R37.1, U8.EN, U8.VIN@1, U8.VIN@2
- net GND: now also C65.-, C66.2, C67.2, C68.1, C69.-, C70.2, C71.2, C72.1, C73.2, C74.2, C75.2, C76.2, C77.-, P1.AGND, P1.PGND, Q5.S, Q6.S, Q7.S, Q8.S, R33.1, R34.1, R35.1, R36.1, R38.2, SV1.1, SW1.P, SW1.P1, SW2.P, SW2.P1, U8.GND, U8.GND1, X5-1.KL, X5-10.KL, X5-19.KL, X5-4.KL
Other:
- note added: "FAN"
- note added: "FILTERING"
- note added: "Floating / GND"
- note added: "ICSP"
- note added: "LDO: 5V -> 3.3V"
- note added: "Normal: floating. Pressed: GND"
- note added: "RESET"
- note added: "RGB STRIP"
- note added: "SMPS module: 24V -> 5V"
- note added: "Seems connected to N-trans gate via 410Ohm"
- note added: "USER INTERFACE"
- note removed: "TODO: - SMPS: 24V -> 5V - LDO: 5V -> 3V3"

Commit message: More schematic work
Parts:
- added C78, C79, C80: (no value), rcl:C-EUC0402
- added D1, D2: BAT60A, diode:BAT60J
- added J6: USB-C-FEMALE, robbe:USB-C-FEMALE
- added Q9: PFETSM, robbe:PFETSM
- added R41, R42, R43, R44, R45, R46, R47: (no value), rcl:R-US_R0402
- added X6: HB THERM, JST_XH:JST-XH-02-PIN-LONG-PAD
Connections:
- new net DN: C78.1, IC1.P0[30]/USB_DMINUS, R45.1
- new net DP: C79.1, IC1.P0[29]/USB_DPLUS, R44.1, R46.2
- new net HB_TEMP: C80.2, IC1.P0[23]/AD0[0]/I2SRX_CLK/CAP3[0], R47.1, X6-2.S
- new net LCD_CS_N: IC1.P0[16]/RXD1/SSEL0/SSEL, X5-14.KL
- new net LCD_D/C_N: IC1.P1[28]/MCOA2/PCAP1[0]/MAT0[0], X5-16.KL
- new net LCD_PWR_EN: IC1.P1[29]/MCOB2/PCAP1[1]/MAT0[1], X5-17.KL
- new net LCD_RES_N: IC1.P1[30]/VBUS/AD0[4], X5-18.KL
- new net LCD_SCLK: IC1.P0[15]/TXD1/SCK0/SCK, X5-13.KL
- new net LCD_SDIN: IC1.P0[18]/DCD1/MOSI0/MOSI, X5-15.KL
- new net N$59: D1.A, P1.VOUT, R37.1
- new net N$60: Q9.S, R46.1
- new net ROT_B: IC1.P1[22]/MCOB0/USB_PWRD/MAT1[0], R42.1
- new net SD_CLK: IC1.P0[7]/I2STX_CLK/SCK1/MAT2[1], X5-5.KL
- new net SD_CS: IC1.P0[6]/I2SRX_SDA/SSEL1/MAT2[0], X5-6.KL
- new net SD_MISO: IC1.P0[8]/I2STX_WS/MISO1/MAT2[2], X5-8.KL
- new net SD_MOSI: IC1.P0[9]/I2STX_SDA/MOSI1/MAT2[3], X5-7.KL
- new net USB_CONNECT: IC1.P2[9]/USB_CONNECT/RXD2/ENET_MDIO, Q9.G
- new net USB_DN: J6.D-A, J6.D-B, R45.2
- new net USB_DP: J6.D+A, J6.D+B, R44.2
- new net VUSB: D2.A, J6.VBUS@1, J6.VBUS@2, J6.VBUS@3, J6.VBUS@4
- net +3V3: now also Q9.D, R41.2, R42.2, R43.2, R47.2
- net +5V: now also D1.C, D2.C; no longer P1.VOUT, R37.1
- net BTN: now also IC1.P1[23]/MCI1/PWM1[4]/MISO0, R43.1
- net BUZZER_GATE: now also IC1.P1[24]/MCI2/PWM1[5]/MOSI0
- net GND: now also C78.2, C79.2, C80.1, J6.GND@1, J6.GND@2, J6.GND@3, J6.GND@4, J6.SHIELDA, J6.SHIELDB, X6-1.S
- net RGB_B: now also IC1.P1[20]/MCI0/PWM1[2]/SCK0; no longer IC1.P1[21]/MCABORT/PWM1[3]/SSEL0
- net RGB_G: now also IC1.P1[19]/MCOA0/USB_PPWR/CAP1[1]; no longer IC1.P1[20]/MCI0/PWM1[2]/SCK0
- net ROT_A: now also IC1.P1[21]/MCABORT/PWM1[3]/SSEL0, R41.1
- net X_END: now also IC1.P1[25]/MCOA1/MAT1[1]; no longer IC1.P1[24]/MCI2/PWM1[5]/MOSI0
- net Z_END: now also IC1.P1[27]/CLKOUT/USB_OVRCR/CAP0[1]; no longer IC1.P1[28]/MCOA2/PCAP1[0]/MAT0[0]
Other:
- note added: "All LCD pins seem to have the right amount of pull-ups and pull-downs. Nice."
- note added: "Already has 5k pullup"
- note added: "CONNECTOR"
- note added: "DATA"
- note added: "EXTRUDER"
- note added: "HEATED BED"
- note added: "ROTARY ENCODER"
- note added: "TEMPERATURE"
- note added: "USB"

Commit message: More stuff
Parts:
- added C81: (no value), rcl:CPOL-EU150CLZ-0810
- added J7: 1744428-4, robbe:1744428-4
- added J8: 282814-4, robbe:282814-4
Connections:
- new net N$61: J7.3, J7.4, Q4.D
- net +24V: now also C81.+, J7.1, J7.2, J8.1, J8.3
- net GND: now also C81.-, J8.2, J8.4
Other:
- note added: "24V INPUT"
- note added: "SMPS MODULE: 24V -> 5V"
- note removed: "SMPS module: 24V -> 5V"
- moved on the sheet: R41, R42, R43, X5-1, X5-10, X5-11, X5-12, X5-13, X5-14, X5-15, X5-16, X5-17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

Commit message: Schematic finished!
Parts:
- added C82, C83, C85, C86, C87, C88, C89: (no value), rcl:C-EUC0402
- added C84: (no value), rcl:CPOL-EU150CLZ-0810
- added J10: B4B-XH-A(LF)(SN), B4B-XH-A_LF__SN_:B4B-XH-A(LF)(SN)
- added J9: 1-281742-2, robbe:1-281742-2
- added LED1, LED2, LED3, LED4, LED5, LED6, LED7: (no value), led:LEDCHIP-LED0603
- added Q10, Q11: SSM3K329R,LF, robbe:SSM3K329R,LF
- added R48, R49, R50, R51, R52, R53, R54, R55: (no value), rcl:R-US_R0402
- added U9: PCA9306DCTR, PCA9306:PCA9306DCTR
- added X7: SENSER, JST_XH:JST-XH-03-PIN-LONG-PAD
Connections:
- new net EXTR_HEATER: J9.12, J9.13, J9.14, J9.15, J9.16, Q3.D
- new net EXTR_TEMP: C83.1, IC1.P0[24]/AD0[1]/I2SRX_WS/CAP3[1], J9.20
- new net E_A1: J9.3, U4.OA1
- new net E_A2: J9.5, U4.OA2
- new net E_B1: J9.4, U4.OB1
- new net E_B2: J9.6, U4.OB2
- new net FAN1: J9.22, Q10.D
- new net FAN1_EN: IC1.P2[11]/EINT1/I2STX_CLK, Q10.G, R48.2
- new net FAN2: J9.21, Q11.D
- new net FAN2_EN: IC1.P2[12]/EINT2/I2STX_WS, Q11.G, R49.2
- new net LED1: IC1.P0[25]/AD0[2]/I2SRX_SDA/TXD3, LED1.A
- new net LED2: IC1.P0[26]/AD0[3]/AOUT/RXD3, LED2.A
- new net LED3: IC1.P0[27]/SDA0/USB_SDA, LED3.A
- new net LED4: IC1.P0[28]/SCL0/USB_SCL, LED4.A
- new net N$62: C85.2, R50.2, X7-3.S
- new net N$63: C86.2, R51.2, X7-1.S
- new net N$64: J10.3, U9.SCL2
- new net N$65: J10.4, U9.SDA2
- new net SCL: IC1.P0[1]/TD1/RXD3/SCL1, R55.1, U9.SCL1
- new net SDA: IC1.P0[0]/RD1/TXD3/SDA1, R54.1, U9.SDA1
- new net SENSER_CONN: IC1.P3[25]/MAT0[0]/PWM1[2], R50.1, R52.1
- new net SENSER_PROBE: IC1.P3[26]/STCLK/MAT0[1]/PWM1[3], R51.1, R53.1
- net +24V: now also C84.+, J9.10, J9.11, J9.7, J9.8, J9.9
- net +3V3: now also C82.2, C87.2, J9.19, LED5.A, R52.2, R53.2, R54.2, R55.2, U9.VREF1
- net +5V: now also C88.2, C89.2, J10.1, U9.EN, U9.VREF2
- net EXTR_HEATER_EN: now also LED6.A
- net GND: now also C82.1, C83.2, C84.-, C85.1, C86.1, C87.1, C88.1, C89.1, J10.2, J9.17, J9.18, LED1.C, LED2.C, LED3.C, LED4.C, LED5.C, LED6.C, LED7.C, Q10.S, Q11.S, R48.1, R49.1, U9.GND, X7-2.S
- net HB_EN: now also LED7.A
Other:
- note added: "AUTOMATIC BED LEVELING"
- note added: "EXTRUDER CABLE"
- note added: "FAN CONTROL"
- note added: "FILAMENT SENSOR"
- note added: "LEDS"
- note added: "SENSER"
- note removed: "EXTRUDER"
- note removed: "TODO: E-axis connections"

Commit message: Started on board
Parts:
- added MNT1, MNT2, MNT3, MNT4, MNT5: MOUNT, robbe:MOUNT
- J1: value B4B-XH-A(LF)(SN) -> X-AXIS
- J2: value B4B-XH-A(LF)(SN) -> Y-AXIS
- J3: value B4B-XH-A(LF)(SN) -> Z_AXIS
- J5: value B4B-XH-A(LF)(SN) -> RGB LED
- Q1: value (none) -> 12MHz; device crystal:CRYSTALHC49UP -> robbe:CRYSTAL; FREQ 12MHz -> (none); MPN J49SMH-A-G-G-K-12M0 -> CX3225SB12000H0PSTC1
- Q2: value (none) -> 25MHz; device crystal:CRYSTALHC49UP -> robbe:CRYSTAL; FREQ 25MHz -> (none); MPN J49SMH-A-G-G-K-12M0 -> CX3225SB25000H0FLJCC
- X2: value X-AXIS -> Y-AXIS
- X3: value X-AXIS -> Z-AXIS
- X5: value UI -> LCD
Connections:
- removed net N$47: C53.1, Q2.2, R19.2, U5.XTAL2
- new net N$67: C53.1, Q2.1, R19.2, U5.XTAL2
- net GND: now also MNT1.MNT, MNT2.MNT, MNT3.MNT, MNT4.MNT, MNT5.MNT, Q1.2, Q2.2
- net N$1: now also Q1.1; no longer Q1.2
- net N$2: now also Q1.3; no longer Q1.1
- net N$48: now also Q2.3; no longer Q2.1
Other:
- note added: "MOUNTING"
- moved on the sheet: C2, C47, C48, C49, C50, C51, C52, C54, C85, C86, J4, R13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

Commit message: Minor schematic improvements and initial routing work
Parts:
- C1, C10, C11, C12, C13, C14, C15, C17, C18, C19, C2, C20, C21, C22, C23, C24, C26, C27, C28, C29, C3, C30, C31, C32, C33, C35, C36, C37, C38, C39, C4, C40, C41, C42, C43, C44, C45, C46, C47, C48, C49, C5, C50, C51, C52, C53, C54, C55, C56, C57, C58, C59, C6, C60, C61, C62, C63, C64, C68, C72, C78, C79, C8, C80, C82, C83, C85, C86, C87, C88, C89, C9: value (none) -> C; device rcl:C-EUC0402 -> robbe:C
