File: board/olchanowski.sch (EAGLE design)
At the start: 201 parts, among them IC1 LPC1768, J1 X-AXIS, J10 B4B-XH-A(LF)(SN), J2 Y-AXIS, J3 Z_AXIS, J4 ARJM11D7-009-AB-ER2-T, J5 RGB LED, J6 USB-C-FEMALE, J7 1744428-4, J8 282814-4, J9 1-281742-2, P1 TPSM53602, Q1 12MHz, Q10 SSM3K329R,LF, Q11 SSM3K329R,LF, Q2 25MHz, Q3 SIJA58DP, Q4 SIJA58DP, Q5 SSM3K329R,LF, Q6 SSM3K329R,LF, Q7 SSM3K329R,LF, Q8 SSM3K329R,LF, Q9 PFETSM, SW1 SPST-2-4PIN, SW2 SPST-2-4PIN, U1 TMC2209-LA, U2 TMC2209-LA, U3 TMC2209-LA, U4 TMC2209-LA, U5 LAN8720, U6 74HC1G04, U7 LM5111, U8 NCP5661-0, U9 PCA9306DCTR, X1 X-AXIS, X2 Y-AXIS, X3 Z-AXIS, X4 FAN, X5 LCD, X6 HB THERM, X7 SENSER

Commit message: Component placement
Connections:
- removed net ROT_B\: X5-12.KL
- net ROT_B: now also X5-12.KL

Commit message: More routing
Parts:
- removed C84: (no value), rcl:CPOL-EU150CLZ-0810
- added C90, C91: C, robbe:C
Connections:
- net +24V: no longer C84.+
- net +3V3: now also C90.2, C91.2
- net +5V: no longer C70.1, C71.1, C72.2
- net BTN: now also IC1.P4[29]/TX_MCLK/MAT2[1]/RXD3; no longer IC1.P1[23]/MCI1/PWM1[4]/MISO0
- net BUZZER_GATE: now also IC1.P4[28]/RX_MCLK/MAT2[0]/TXD3; no longer IC1.P1[24]/MCI2/PWM1[5]/MOSI0
- net GND: now also C90.1, C91.1; no longer C84.-
- net N$59: now also C70.1, C71.1, C72.2
Other:
- moved on the sheet: C58, C60, C61, C69, C70, C71, C72, C82, C83, D1, J9

Commit message: Routing
Connections:
- net TMC_DIR_X: now also IC1.P0[10]/TXD2/SDA2/MAT3[0]; no longer IC1.P0[5]/I2SRX_WS/TD2/CAP2[1]
- net TMC_DIR_Y: now also IC1.P0[5]/I2SRX_WS/TD2/CAP2[1]; no longer IC1.P0[11]/RXD2/SCL2/MAT3[1]
- net TMC_ENN_X: now also IC1.P0[11]/RXD2/SCL2/MAT3[1]; no longer IC1.P0[4]/I2SRX_CLK/RD2/CAP2[0]
- net TMC_ENN_Y: now also IC1.P0[4]/I2SRX_CLK/RD2/CAP2[0]; no longer IC1.P0[10]/TXD2/SDA2/MAT3[0]
- net TMC_STEP_X: now also IC1.P2[2]/PWM1[3]/CTS1/TRACEDATA[3]; no longer IC1.P2[0]/PWM1[1]/TXD1
- net TMC_STEP_Z: now also IC1.P2[0]/PWM1[1]/TXD1; no longer IC1.P2[2]/PWM1[3]/CTS1/TRACEDATA[3]
Changed lines of the file:
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@@
 <?xml version="1.0" encoding="utf-8"?>
 <!DOCTYPE eagle SYSTEM "eagle.dtd">
-<eagle version="9.6.0">
+<eagle version="9.6.1">
 <drawing>
 <settings>
@@
 </segment>
 </net>
-<net name="TMC_STEP_X" class="0">
-<segment>
-<wire x1="137.16" y1="175.26" x2="160.02" y2="175.26" width="0.1524" layer="91"/>
-<label x="139.7" y="175.26" size="1.778" layer="95"/>
-<pinref part="IC1" gate="G$1" pin="P2[0]/PWM1[1]/TXD1"/>
-</segment>
-</net>
 <net name="TMC_STEP_Y" class="0">
 <segment>
@@
 </segment>
 </net>
-<net name="TMC_STEP_Z" class="0">
-<segment>
-<wire x1="137.16" y1="170.18" x2="160.02" y2="170.18" width="0.1524" layer="91"/>
-<label x="139.7" y="170.18" size="1.778" layer="95"/>
-<pinref part="IC1" gate="G$1" pin="P2[2]/PWM1[3]/CTS1/TRACEDATA[3]"/>
-</segment>
-</net>
 <net name="TMC_STEP_E" class="0">
 <segment>
@@
 </segment>
 </net>
-<net name="TMC_DIR_X" class="0">
-<segment>
-<pinref part="IC1" gate="G$1" pin="P0[5]/I2SRX_WS/TD2/CAP2[1]"/>
-<wire x1="48.26" y1="226.06" x2="30.48" y2="226.06" width="0.1524" layer="91"/>
-<label x="30.48" y="226.06" size="1.778" layer="95"/>
-</segment>
-</net>
-<net name="TMC_DIR_Y" class="0">
-<segment>
-<pinref part="IC1" gate="G$1" pin="P0[11]/RXD2/SCL2/MAT3[1]"/>
-<wire x1="48.26" y1="210.82" x2="30.48" y2="210.82" width="0.1524" layer="91"/>
-<label x="30.48" y="210.82" size="1.778" layer="95"/>
-</segment>
-</net>
 <net name="TMC_DIR_Z" class="0">
 <segment>
@@
 <wire x1="48.26" y1="190.5" x2="30.48" y2="190.5" width="0.1524" layer="91"/>
 <label x="30.48" y="190.5" size="1.778" layer="95"/>
-</segment>
-</net>
-<net name="TMC_ENN_X" class="0">
-<segment>
-<pinref part="IC1" gate="G$1" pin="P0[4]/I2SRX_CLK/RD2/CAP2[0]"/>
-<wire x1="48.26" y1="228.6" x2="30.48" y2="228.6" width="0.1524" layer="91"/>
-<label x="30.48" y="228.6" size="1.778" layer="95"/>
-</segment>
-</net>
-<net name="TMC_ENN_Y" class="0">
-<segment>
-<pinref part="IC1" gate="G$1" pin="P0[10]/TXD2/SDA2/MAT3[0]"/>
-<wire x1="48.26" y1="213.36" x2="30.48" y2="213.36" width="0.1524" layer="91"/>
-<label x="30.48" y="213.36" size="1.778" layer="95"/>
 </segment>
 </net>
@@
 </segment>
 </net>
+<net name="TMC_DIR_Y" class="0">
+<segment>
+<wire x1="48.26" y1="226.06" x2="30.48" y2="226.06" width="0.1524" layer="91"/>
+<label x="30.48" y="226.06" size="1.778" layer="95"/>
+<pinref part="IC1" gate="G$1" pin="P0[5]/I2SRX_WS/TD2/CAP2[1]"/>
+</segment>
+</net>
+<net name="TMC_ENN_Y" class="0">
+<segment>
+<wire x1="48.26" y1="228.6" x2="30.48" y2="228.6" width="0.1524" layer="91"/>
+<label x="30.48" y="228.6" size="1.778" layer="95"/>
+<pinref part="IC1" gate="G$1" pin="P0[4]/I2SRX_CLK/RD2/CAP2[0]"/>
+</segment>
+</net>
+<net name="TMC_STEP_Z" class="0">
+<segment>
+<wire x1="137.16" y1="175.26" x2="160.02" y2="175.26" width="0.1524" layer="91"/>
+<label x="139.7" y="175.26" size="1.778" layer="95"/>
+<pinref part="IC1" gate="G$1" pin="P2[0]/PWM1[1]/TXD1"/>
+</segment>
+</net>
+<net name="TMC_STEP_X" class="0">
+<segment>
+<wire x1="137.16" y1="170.18" x2="160.02" y2="170.18" width="0.1524" layer="91"/>
+<label x="139.7" y="170.18" size="1.778" layer="95"/>
+<pinref part="IC1" gate="G$1" pin="P2[2]/PWM1[3]/CTS1/TRACEDATA[3]"/>
+</segment>
+</net>
+<net name="TMC_DIR_X" class="0">
+<segment>
+<wire x1="48.26" y1="213.36" x2="30.48" y2="213.36" width="0.1524" layer="91"/>
+<label x="30.48" y="213.36" size="1.778" layer="95"/>
+<pinref part="IC1" gate="G$1" pin="P0[10]/TXD2/SDA2/MAT3[0]"/>
+</segment>
+</net>
+<net name="TMC_ENN_X" class="0">
+<segment>
+<wire x1="48.26" y1="210.82" x2="30.48" y2="210.82" width="0.1524" layer="91"/>
+<label x="30.48" y="210.82" size="1.778" layer="95"/>
+<pinref part="IC1" gate="G$1" pin="P0[11]/RXD2/SCL2/MAT3[1]"/>
+</segment>
+</net>

Commit message: First rev done and ordered!
Parts:
- added R56: (no value), rcl:R-US_R0402
Connections:
- removed net ENET_TXD_EN: IC1.P1[4]/ENET_TX_EN
- new net N$47: IC1.P0[10]/TXD2/SDA2/MAT3[0], R56.1
- net ENET_TX_EN: now also IC1.P1[4]/ENET_TX_EN
- net TMC_DIR_X: now also IC1.P1[24]/MCI2/PWM1[5]/MOSI0; no longer IC1.P0[10]/TXD2/SDA2/MAT3[0]
- net TMC_ENN_X: now also IC1.P1[23]/MCI1/PWM1[4]/MISO0; no longer IC1.P0[11]/RXD2/SCL2/MAT3[1]
- net TMC_UART: now also IC1.P0[11]/RXD2/SCL2/MAT3[1], R56.2

Commit message: Added order list
Parts:
- J10: AXIS X -> (none)
- U5: MPN (none) -> LAN8720A-CP-TR-ABC
Changed lines of the file:
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@@
 <part name="GND38" library="supply1" library_urn="urn:adsk.eagle:library:371" deviceset="GND" device=""/>
 <part name="FRAME4" library="frames" library_urn="urn:adsk.eagle:library:229" deviceset="A4L-LOC" device=""/>
-<part name="U5" library="microchip-smsc-lan8720" deviceset="LAN8720" device=""/>
+<part name="U5" library="microchip-smsc-lan8720" deviceset="LAN8720" device="">
+<attribute name="MPN" value="LAN8720A-CP-TR-ABC"/>
+</part>
 <part name="J4" library="robbe" deviceset="ARJM11D7-009-AB-ER2-T" device="">
 <attribute name="MPN" value="ARJM11D7-009-AB-ER2-T"/>
@@
 <attribute name="R" value="10k"/>
 </part>
-<part name="J10" library="B4B-XH-A_LF__SN_" deviceset="B4B-XH-A(LF)(SN)" device="">
-<attribute name="AXIS" value="X"/>
-</part>
+<part name="J10" library="B4B-XH-A_LF__SN_" deviceset="B4B-XH-A(LF)(SN)" device=""/>
 <part name="GND128" library="supply1" library_urn="urn:adsk.eagle:library:371" deviceset="GND" device=""/>
 <part name="C88" library="robbe" deviceset="C" device="">
@@
 <attribute name="NAME" x="45.72" y="157.48" size="1.778" layer="95"/>
 <attribute name="VALUE" x="45.72" y="154.94" size="1.778" layer="96"/>
+<attribute name="MPN" x="63.5" y="129.54" size="1.778" layer="96" display="off"/>
 </instance>
 <instance part="J4" gate="G$1" x="231.14" y="121.92" smashed="yes">
@@
 </instance>
 <instance part="J10" gate="G$1" x="38.1" y="53.34" smashed="yes" rot="MR180">
-<attribute name="NAME" x="42.915890625" y="58.677159375" size="1.780209375" layer="95" rot="MR270"/>
-<attribute name="AXIS" x="35.052" y="57.404" size="1.778" layer="96" rot="MR270" display="both"/>
+<attribute name="NAME" x="35.810840625" y="44.947890625" size="1.780209375" layer="95" rot="MR180"/>
 </instance>
 <instance part="GND128" gate="1" x="48.26" y="38.1" smashed="yes">

Commit message: Update Cap P/N
Parts:
- C12, C21, C3, C30: MPN CC0402KRX7R9BB222 -> GRM155R71H223KA12J
Changed lines of the file:
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@@
 <?xml version="1.0" encoding="utf-8"?>
 <!DOCTYPE eagle SYSTEM "eagle.dtd">
-<eagle version="9.6.0">
+<eagle version="9.6.1">
 <drawing>
 <settings>
@@
 <grid distance="0.1" unitdist="inch" unit="inch" style="lines" multiple="1" display="no" altdistance="0.01" altunitdist="inch" altunit="inch"/>
 <layers>
-<layer number="1" name="Top" color="4" fill="1" visible="yes" active="no"/>
-<layer number="2" name="Route2" color="16" fill="1" visible="yes" active="no"/>
-<layer number="3" name="Route3" color="17" fill="1" visible="yes" active="no"/>
-<layer number="4" name="Route4" color="18" fill="1" visible="yes" active="no"/>
-<layer number="5" name="Route5" color="19" fill="1" visible="yes" active="no"/>
-<layer number="6" name="Route6" color="25" fill="1" visible="yes" active="no"/>
-<layer number="7" name="Route7" color="26" fill="1" visible="yes" active="no"/>
-<layer number="8" name="Route8" color="27" fill="1" visible="yes" active="no"/>
-<layer number="9" name="Route9" color="28" fill="1" visible="yes" active="no"/>
-<layer number="10" name="Route10" color="29" fill="1" visible="yes" active="no"/>
-<layer number="11" name="Route11" color="30" fill="1" visible="yes" active="no"/>
-<layer number="12" name="Route12" color="20" fill="1" visible="yes" active="no"/>
-<layer number="13" name="Route13" color="21" fill="1" visible="yes" active="no"/>
-<layer number="14" name="Route14" color="22" fill="1" visible="yes" active="no"/>
-<layer number="15" name="Route15" color="23" fill="1" visible="yes" active="no"/>
-<layer number="16" name="Bottom" color="1" fill="1" visible="yes" active="no"/>
-<layer number="17" name="Pads" color="2" fill="1" visible="yes" active="no"/>
-<layer number="18" name="Vias" color="2" fill="1" visible="yes" active="no"/>
-<layer number="19" name="Unrouted" color="6" fill="1" visible="yes" active="no"/>
-<layer number="20" name="Dimension" color="24" fill="1" visible="yes" active="no"/>
-<layer number="21" name="tPlace" color="7" fill="1" visible="yes" active="no"/>
-<layer number="22" name="bPlace" color="7" fill="1" visible="yes" active="no"/>
-<layer number="23" name="tOrigins" color="15" fill="1" visible="yes" active="no"/>
-<layer number="24" name="bOrigins" color="15" fill="1" visible="yes" active="no"/>
-<layer number="25" name="tNames" color="7" fill="1" visible="yes" active="no"/>
-<layer number="26" name="bNames" color="7" fill="1" visible="yes" active="no"/>
-<layer number="27" name="tValues" color="7" fill="1" visible="yes" active="no"/>
-<layer number="28" name="bValues" color="7" fill="1" visible="yes" active="no"/>
+<layer number="1" name="Top" color="4" fill="1" visible="no" active="no"/>
+<layer number="2" name="Route2" color="16" fill="1" visible="no" active="no"/>
+<layer number="3" name="Route3" color="17" fill="1" visible="no" active="no"/>
+<layer number="4" name="Route4" color="18" fill="1" visible="no" active="no"/>
+<layer number="5" name="Route5" color="19" fill="1" visible="no" active="no"/>
+<layer number="6" name="Route6" color="25" fill="1" visible="no" active="no"/>
+<layer number="7" name="Route7" color="26" fill="1" visible="no" active="no"/>
+<layer number="8" name="Route8" color="27" fill="1" visible="no" active="no"/>
+<layer number="9" name="Route9" color="28" fill="1" visible="no" active="no"/>
+<layer number="10" name="Route10" color="29" fill="1" visible="no" active="no"/>
+<layer number="11" name="Route11" color="30" fill="1" visible="no" active="no"/>
+<layer number="12" name="Route12" color="20" fill="1" visible="no" active="no"/>
+<layer number="13" name="Route13" color="21" fill="1" visible="no" active="no"/>
+<layer number="14" name="Route14" color="22" fill="1" visible="no" active="no"/>
+<layer number="15" name="Route15" color="23" fill="1" visible="no" active="no"/>
+<layer number="16" name="Bottom" color="1" fill="1" visible="no" active="no"/>
+<layer number="17" name="Pads" color="2" fill="1" visible="no" active="no"/>
+<layer number="18" name="Vias" color="2" fill="1" visible="no" active="no"/>
+<layer number="19" name="Unrouted" color="6" fill="1" visible="no" active="no"/>
+<layer number="20" name="Dimension" color="24" fill="1" visible="no" active="no"/>
+<layer number="21" name="tPlace" color="7" fill="1" visible="no" active="no"/>
+<layer number="22" name="bPlace" color="7" fill="1" visible="no" active="no"/>
+<layer number="23" name="tOrigins" color="15" fill="1" visible="no" active="no"/>
+<layer number="24" name="bOrigins" color="15" fill="1" visible="no" active="no"/>
+<layer number="25" name="tNames" color="7" fill="1" visible="no" active="no"/>
+<layer number="26" name="bNames" color="7" fill="1" visible="no" active="no"/>
+<layer number="27" name="tValues" color="7" fill="1" visible="no" active="no"/>
+<layer number="28" name="bValues" color="7" fill="1" visible="no" active="no"/>
 <layer number="29" name="tStop" color="7" fill="3" visible="no" active="no"/>
 <layer number="30" name="bStop" color="7" fill="6" visible="no" active="no"/>
@@
 <layer number="35" name="tGlue" color="7" fill="4" visible="no" active="no"/>
 <layer number="36" name="bGlue" color="7" fill="5" visible="no" active="no"/>
-<layer number="37" name="tTest" color="7" fill="1" visible="yes" active="no"/>
-<layer number="38" name="bTest" color="7" fill="1" visible="yes" active="no"/>
+<layer number="37" name="tTest" color="7" fill="1" visible="no" active="no"/>
+<layer number="38" name="bTest" color="7" fill="1" visible="no" active="no"/>
 <layer number="39" name="tKeepout" color="4" fill="11" visible="no" active="no"/>
 <layer number="40" name="bKeepout" color="1" fill="11" visible="no" active="no"/>
@@
 <layer number="44" name="Drills" color="7" fill="1" visible="no" active="no"/>
 <layer number="45" name="Holes" color="7" fill="1" visible="no" active="no"/>
-<layer number="46" name="Milling" color="3" fill="1" visible="yes" active="no"/>
-<layer number="47" name="Measures" color="7" fill="1" visible="yes" active="no"/>
-<layer number="48" name="Document" color="7" fill="1" visible="yes" active="no"/>
-<layer number="49" name="Reference" color="7" fill="1" visible="yes" active="no"/>
-<layer number="50" name="dxf" color="7" fill="1" visible="yes" active="no"/>
-<layer number="51" name="tDocu" color="7" fill="1" visible="yes" active="no"/>
-<layer number="52" name="bDocu" color="7" fill="1" visible="yes" active="no"/>
-<layer number="53" name="tGND_GNDA" color="7" fill="9" visible="yes" active="no"/>
-<layer number="54" name="bGND_GNDA" color="1" fill="9" visible="yes" active="no"/>
-<layer number="56" name="wert" color="7" fill="1" visible="yes" active="no"/>
-<layer number="57" name="tCAD" color="7" fill="1" visible="yes" active="no"/>
-<layer number="58" name="bCAD" color="11" fill="1" visible="yes" active="no"/>
-<layer number="59" name="tCarbon" color="7" fill="1" visible="yes" active="no"/>
-<layer number="60" name="bCarbon" color="7" fill="1" visible="yes" active="no"/>
+<layer number="46" name="Milling" color="3" fill="1" visible="no" active="no"/>
+<layer number="47" name="Measures" color="7" fill="1" visible="no" active="no"/>
+<layer number="48" name="Document" color="7" fill="1" visible="no" active="no"/>
+<layer number="49" name="Reference" color="7" fill="1" visible="no" active="no"/>
+<layer number="50" name="dxf" color="7" fill="1" visible="no" active="no"/>
+<layer number="51" name="tDocu" color="7" fill="1" visible="no" active="no"/>
+<layer number="52" name="bDocu" color="7" fill="1" visible="no" active="no"/>
+<layer number="53" name="tGND_GNDA" color="7" fill="9" visible="no" active="no"/>
+<layer number="54" name="bGND_GNDA" color="1" fill="9" visible="no" active="no"/>
+<layer number="56" name="wert" color="7" fill="1" visible="no" active="no"/>
+<layer number="57" name="tCAD" color="7" fill="1" visible="no" active="no"/>
+<layer number="58" name="bCAD" color="11" fill="1" visible="no" active="no"/>
+<layer number="59" name="tCarbon" color="7" fill="1" visible="no" active="no"/>
+<layer number="60" name="bCarbon" color="7" fill="1" visible="no" active="no"/>
 <layer number="88" name="SimResults" color="9" fill="1" visible="yes" active="yes"/>
 <layer number="89" name="SimProbes" color="9" fill="1" visible="yes" active="yes"/>
@@
 </spice>
 <attribute name="C" value="22n"/>
-<attribute name="MPN" value="CC0402KRX7R9BB222"/>
+<attribute name="MPN" value="GRM155R71H223KA12J"/>
 </part>
 <part name="C4" library="robbe" deviceset="C" device="">
@@
 </spice>
 <attribute name="C" value="22n"/>
-<attribute name="MPN" value="CC0402KRX7R9BB222"/>
+<attribute name="MPN" value="GRM155R71H223KA12J"/>
 </part>
 <part name="C13" library="robbe" deviceset="C" device="">
@@
 </spice>
 <attribute name="C" value="22n"/>
-<attribute name="MPN" value="CC0402KRX7R9BB222"/>
+<attribute name="MPN" value="GRM155R71H223KA12J"/>
 </part>
 <part name="C22" library="robbe" deviceset="C" device="">
@@
 </spice>
 <attribute name="C" value="22n"/>
-<attribute name="MPN" value="CC0402KRX7R9BB222"/>
+<attribute name="MPN" value="GRM155R71H223KA12J"/>
 </part>
 <part name="C31" library="robbe" deviceset="C" device="">

Commit message: Fix P1 NC/AGND pins
Connections:
- net GND: now also P1.NC
Changed lines of the file:
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@@
 <net name="GND" class="0">
-<segment>
-<pinref part="P1" gate="G$1" pin="PGND"/>
-<wire x1="60.96" y1="119.38" x2="60.96" y2="116.84" width="0.1524" layer="91"/>
-<pinref part="P1" gate="G$1" pin="AGND"/>
-<wire x1="60.96" y1="116.84" x2="63.5" y2="116.84" width="0.1524" layer="91"/>
-<wire x1="63.5" y1="116.84" x2="66.04" y2="116.84" width="0.1524" layer="91"/>
-<wire x1="66.04" y1="116.84" x2="66.04" y2="119.38" width="0.1524" layer="91"/>
-<pinref part="GND88" gate="1" pin="GND"/>
-<wire x1="63.5" y1="114.3" x2="63.5" y2="116.84" width="0.1524" layer="91"/>
-<junction x="63.5" y="116.84"/>
-</segment>
 <segment>
 <pinref part="R38" gate="G$1" pin="2"/>
@@
 <pinref part="C72" gate="G$1" pin="1"/>
 </segment>
+<segment>
+<pinref part="P1" gate="G$1" pin="NC"/>
+<wire x1="55.88" y1="119.38" x2="55.88" y2="116.84" width="0.1524" layer="91"/>
+<wire x1="55.88" y1="116.84" x2="63.5" y2="116.84" width="0.1524" layer="91"/>
+<pinref part="GND88" gate="1" pin="GND"/>
+<wire x1="63.5" y1="116.84" x2="63.5" y2="114.3" width="0.1524" layer="91"/>
+<pinref part="P1" gate="G$1" pin="PGND"/>
+<wire x1="63.5" y1="119.38" x2="63.5" y2="116.84" width="0.1524" layer="91"/>
+<junction x="63.5" y="116.84"/>
+<pinref part="P1" gate="G$1" pin="AGND"/>
+<wire x1="71.12" y1="119.38" x2="71.12" y2="116.84" width="0.1524" layer="91"/>
+<wire x1="71.12" y1="116.84" x2="63.5" y2="116.84" width="0.1524" layer="91"/>
+</segment>
 </net>
