File: board/olchanowski.sch (EAGLE design)
At the start: 203 parts, among them IC1 LPC1768, J1 X-AXIS, J10 B4B-XH-A(LF)(SN), J2 Y-AXIS, J3 Z_AXIS, J4 ARJM11D7-009-AB-ER2-T, J5 RGB LED, J6 USB-C-FEMALE, J7 1744428-4, J8 282814-4, J9 1-281742-2, P1 TPSM53602, Q1 12MHz, Q10 SSM3K329R,LF, Q11 SSM3K329R,LF, Q2 25MHz, Q3 SIJA58DP, Q4 SIJA58DP, Q5 SSM3K329R,LF, Q6 SSM3K329R,LF, Q7 SSM3K329R,LF, Q8 SSM3K329R,LF, Q9 PFETSM, SW1 SPST-2-4PIN, SW2 SPST-2-4PIN, U1 TMC2209-LA, U2 TMC2209-LA, U3 TMC2209-LA, U4 TMC2209-LA, U5 LAN8720, U6 74HC1G04, U7 LM5111, U8 NCP5661-0, U9 PCA9306DCTR, X1 X-AXIS, X2 Y-AXIS, X3 Z-AXIS, X4 FAN, X5 LCD, X6 HB THERM, X7 SENSER

Commit message: Fix Stepper connector pinout
Connections:
- removed net N$28: J3.1, U3.OA1
- removed net N$30: J3.3, U3.OA2
- removed net N$31: J3.4, U3.OB2
- new net N$66: J1.4, U1.OA2
- new net N$68: J1.3, U1.OA1
- new net N$70: J1.1, U1.OB2
- net E_A1: now also J9.4; no longer J9.3
- net E_B1: now also J9.3; no longer J9.4
- net N$10: now also J2.3, U2.OA1; no longer J1.3, U1.OA2
- net N$11: now also J2.4, U2.OA2; no longer J1.4, U1.OB2
- net N$18: now also J3.1, U3.OB2; no longer J2.1, U2.OA1
- net N$20: now also J3.3, U3.OA1; no longer J2.3, U2.OA2
- net N$21: now also J3.4, U3.OA2; no longer J2.4, U2.OB2
- net N$8: now also J2.1, U2.OB2; no longer J1.1, U1.OA1
Changed lines of the file:
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@@
 </segment>
 </net>
-<net name="N$8" class="0">
-<segment>
-<pinref part="J1" gate="G$1" pin="1"/>
-<wire x1="99.06" y1="119.38" x2="99.06" y2="114.3" width="0.1524" layer="91"/>
-<pinref part="U1" gate="G$1" pin="OA1"/>
-<wire x1="99.06" y1="114.3" x2="93.98" y2="114.3" width="0.1524" layer="91"/>
-</segment>
-</net>
-<net name="N$9" class="0">
-<segment>
-<pinref part="J1" gate="G$1" pin="2"/>
-<wire x1="101.6" y1="119.38" x2="101.6" y2="109.22" width="0.1524" layer="91"/>
-<pinref part="U1" gate="G$1" pin="OB1"/>
-<wire x1="101.6" y1="109.22" x2="93.98" y2="109.22" width="0.1524" layer="91"/>
-</segment>
-</net>
-<net name="N$10" class="0">
-<segment>
-<pinref part="J1" gate="G$1" pin="3"/>
-<wire x1="104.14" y1="119.38" x2="104.14" y2="116.84" width="0.1524" layer="91"/>
-<wire x1="104.14" y1="116.84" x2="93.98" y2="116.84" width="0.1524" layer="91"/>
-<pinref part="U1" gate="G$1" pin="OA2"/>
-</segment>
-</net>
-<net name="N$11" class="0">
-<segment>
-<pinref part="U1" gate="G$1" pin="OB2"/>
-<wire x1="93.98" y1="106.68" x2="106.68" y2="106.68" width="0.1524" layer="91"/>
-<pinref part="J1" gate="G$1" pin="4"/>
-<wire x1="106.68" y1="106.68" x2="106.68" y2="119.38" width="0.1524" layer="91"/>
-</segment>
-</net>
 <net name="N$12" class="0">
 <segment>
@@
 </segment>
 </net>
-<net name="N$18" class="0">
-<segment>
-<pinref part="J2" gate="G$1" pin="1"/>
-<wire x1="218.44" y1="119.38" x2="218.44" y2="114.3" width="0.1524" layer="91"/>
-<pinref part="U2" gate="G$1" pin="OA1"/>
-<wire x1="218.44" y1="114.3" x2="213.36" y2="114.3" width="0.1524" layer="91"/>
-</segment>
-</net>
-<net name="N$19" class="0">
-<segment>
-<pinref part="J2" gate="G$1" pin="2"/>
-<wire x1="220.98" y1="119.38" x2="220.98" y2="109.22" width="0.1524" layer="91"/>
-<pinref part="U2" gate="G$1" pin="OB1"/>
-<wire x1="220.98" y1="109.22" x2="213.36" y2="109.22" width="0.1524" layer="91"/>
-</segment>
-</net>
-<net name="N$20" class="0">
-<segment>
-<pinref part="J2" gate="G$1" pin="3"/>
-<wire x1="223.52" y1="119.38" x2="223.52" y2="116.84" width="0.1524" layer="91"/>
-<wire x1="223.52" y1="116.84" x2="213.36" y2="116.84" width="0.1524" layer="91"/>
-<pinref part="U2" gate="G$1" pin="OA2"/>
-</segment>
-</net>
-<net name="N$21" class="0">
-<segment>
-<pinref part="U2" gate="G$1" pin="OB2"/>
-<wire x1="213.36" y1="106.68" x2="226.06" y2="106.68" width="0.1524" layer="91"/>
-<pinref part="J2" gate="G$1" pin="4"/>
-<wire x1="226.06" y1="106.68" x2="226.06" y2="119.38" width="0.1524" layer="91"/>
-</segment>
-</net>
 <net name="N$22" class="0">
 <segment>
@@
 </segment>
 </net>
+<net name="N$66" class="0">
+<segment>
+<pinref part="U1" gate="G$1" pin="OA2"/>
+<wire x1="93.98" y1="116.84" x2="106.68" y2="116.84" width="0.1524" layer="91"/>
+<pinref part="J1" gate="G$1" pin="4"/>
+<wire x1="106.68" y1="116.84" x2="106.68" y2="119.38" width="0.1524" layer="91"/>
+</segment>
+</net>
+<net name="N$68" class="0">
+<segment>
+<pinref part="U1" gate="G$1" pin="OA1"/>
+<wire x1="93.98" y1="114.3" x2="104.14" y2="114.3" width="0.1524" layer="91"/>
+<pinref part="J1" gate="G$1" pin="3"/>
+<wire x1="104.14" y1="114.3" x2="104.14" y2="119.38" width="0.1524" layer="91"/>
+</segment>
+</net>
+<net name="N$69" class="0">
+<segment>
+<pinref part="U1" gate="G$1" pin="OB1"/>
+<wire x1="93.98" y1="109.22" x2="101.6" y2="109.22" width="0.1524" layer="91"/>
+<pinref part="J1" gate="G$1" pin="2"/>
+<wire x1="101.6" y1="109.22" x2="101.6" y2="119.38" width="0.1524" layer="91"/>
+</segment>
+</net>
+<net name="N$70" class="0">
+<segment>
+<pinref part="U1" gate="G$1" pin="OB2"/>
+<wire x1="93.98" y1="106.68" x2="99.06" y2="106.68" width="0.1524" layer="91"/>
+<pinref part="J1" gate="G$1" pin="1"/>
+<wire x1="99.06" y1="106.68" x2="99.06" y2="119.38" width="0.1524" layer="91"/>
+</segment>
+</net>
+<net name="N$8" class="0">
+<segment>
+<pinref part="U2" gate="G$1" pin="OB2"/>
+<pinref part="J2" gate="G$1" pin="1"/>
+<wire x1="213.36" y1="106.68" x2="218.44" y2="106.68" width="0.1524" layer="91"/>
+<wire x1="218.44" y1="106.68" x2="218.44" y2="119.38" width="0.1524" layer="91"/>
+</segment>
+</net>
+<net name="N$9" class="0">
+<segment>
+<pinref part="U2" gate="G$1" pin="OB1"/>
+<wire x1="213.36" y1="109.22" x2="220.98" y2="109.22" width="0.1524" layer="91"/>
+<pinref part="J2" gate="G$1" pin="2"/>
+<wire x1="220.98" y1="109.22" x2="220.98" y2="119.38" width="0.1524" layer="91"/>
+</segment>
+</net>
+<net name="N$10" class="0">
+<segment>
+<pinref part="U2" gate="G$1" pin="OA1"/>
+<wire x1="213.36" y1="114.3" x2="223.52" y2="114.3" width="0.1524" layer="91"/>
+<pinref part="J2" gate="G$1" pin="3"/>
+<wire x1="223.52" y1="114.3" x2="223.52" y2="119.38" width="0.1524" layer="91"/>
+</segment>
+</net>
+<net name="N$11" class="0">
+<segment>
+<pinref part="U2" gate="G$1" pin="OA2"/>
+<wire x1="213.36" y1="116.84" x2="226.06" y2="116.84" width="0.1524" layer="91"/>
+<pinref part="J2" gate="G$1" pin="4"/>
+<wire x1="226.06" y1="116.84" x2="226.06" y2="119.38" width="0.1524" layer="91"/>
+</segment>
+</net>
 </nets>
 </sheet>
@@
 </segment>
 </net>
-<net name="N$28" class="0">
-<segment>
-<pinref part="J3" gate="G$1" pin="1"/>
-<wire x1="99.06" y1="119.38" x2="99.06" y2="114.3" width="0.1524" layer="91"/>
-<pinref part="U3" gate="G$1" pin="OA1"/>
-<wire x1="99.06" y1="114.3" x2="93.98" y2="114.3" width="0.1524" layer="91"/>
-</segment>
-</net>
-<net name="N$29" class="0">
-<segment>
-<pinref part="J3" gate="G$1" pin="2"/>
-<wire x1="101.6" y1="119.38" x2="101.6" y2="109.22" width="0.1524" layer="91"/>
-<pinref part="U3" gate="G$1" pin="OB1"/>
-<wire x1="101.6" y1="109.22" x2="93.98" y2="109.22" width="0.1524" layer="91"/>
-</segment>
-</net>
-<net name="N$30" class="0">
-<segment>
-<pinref part="J3" gate="G$1" pin="3"/>
-<wire x1="104.14" y1="119.38" x2="104.14" y2="116.84" width="0.1524" layer="91"/>
-<wire x1="104.14" y1="116.84" x2="93.98" y2="116.84" width="0.1524" layer="91"/>
-<pinref part="U3" gate="G$1" pin="OA2"/>
-</segment>
-</net>
-<net name="N$31" class="0">
-<segment>
-<pinref part="U3" gate="G$1" pin="OB2"/>
-<wire x1="93.98" y1="106.68" x2="106.68" y2="106.68" width="0.1524" layer="91"/>
-<pinref part="J3" gate="G$1" pin="4"/>
-<wire x1="106.68" y1="106.68" x2="106.68" y2="119.38" width="0.1524" layer="91"/>
-</segment>
-</net>
 <net name="N$32" class="0">
 <segment>
@@
 </segment>
 </net>
+<net name="N$18" class="0">
+<segment>
+<pinref part="U3" gate="G$1" pin="OB2"/>
+<wire x1="93.98" y1="106.68" x2="99.06" y2="106.68" width="0.1524" layer="91"/>
+<pinref part="J3" gate="G$1" pin="1"/>
+<wire x1="99.06" y1="106.68" x2="99.06" y2="119.38" width="0.1524" layer="91"/>
+</segment>
+</net>
+<net name="N$19" class="0">
+<segment>
+<pinref part="U3" gate="G$1" pin="OB1"/>
+<wire x1="93.98" y1="109.22" x2="101.6" y2="109.22" width="0.1524" layer="91"/>
+<pinref part="J3" gate="G$1" pin="2"/>
+<wire x1="101.6" y1="109.22" x2="101.6" y2="119.38" width="0.1524" layer="91"/>
+</segment>
+</net>
+<net name="N$20" class="0">
+<segment>
+<pinref part="U3" gate="G$1" pin="OA1"/>
+<wire x1="93.98" y1="114.3" x2="104.14" y2="114.3" width="0.1524" layer="91"/>
+<pinref part="J3" gate="G$1" pin="3"/>
+<wire x1="104.14" y1="114.3" x2="104.14" y2="119.38" width="0.1524" layer="91"/>
+</segment>
+</net>
+<net name="N$21" class="0">
+<segment>
+<pinref part="U3" gate="G$1" pin="OA2"/>
+<wire x1="93.98" y1="116.84" x2="106.68" y2="116.84" width="0.1524" layer="91"/>
+<pinref part="J3" gate="G$1" pin="4"/>
+<wire x1="106.68" y1="116.84" x2="106.68" y2="119.38" width="0.1524" layer="91"/>
+</segment>
+</net>
 </nets>
 </sheet>
@@
 </segment>
 </net>
-<net name="E_A2" class="0">
-<segment>
-<pinref part="J9" gate="G$1" pin="5"/>
-<wire x1="55.88" y1="127" x2="35.56" y2="127" width="0.1524" layer="91"/>
-<label x="35.56" y="127" size="1.778" layer="95"/>
-</segment>
-</net>
-<net name="E_A1" class="0">
-<segment>
-<pinref part="J9" gate="G$1" pin="3"/>
-<wire x1="55.88" y1="124.46" x2="35.56" y2="124.46" width="0.1524" layer="91"/>
-<label x="35.56" y="124.46" size="1.778" layer="95"/>
-</segment>
-</net>
-<net name="E_B1" class="0">
-<segment>
-<pinref part="J9" gate="G$1" pin="4"/>
-<wire x1="78.74" y1="124.46" x2="101.6" y2="124.46" width="0.1524" layer="91"/>
-<label x="86.36" y="124.46" size="1.778" layer="95"/>
-</segment>
-</net>
-<net name="E_B2" class="0">
-<segment>
-<pinref part="J9" gate="G$1" pin="6"/>
-<wire x1="78.74" y1="127" x2="101.6" y2="127" width="0.1524" layer="91"/>
-<label x="86.36" y="127" size="1.778" layer="95"/>
-</segment>
-</net>
 <net name="EXTR_TEMP" class="0">
 <segment>
@@
 </segment>
 </net>
+<net name="E_B1" class="0">
+<segment>
+<pinref part="J9" gate="G$1" pin="3"/>
+<wire x1="55.88" y1="124.46" x2="43.18" y2="124.46" width="0.1524" layer="91"/>
+<label x="45.72" y="124.46" size="1.778" layer="95"/>
+</segment>
+</net>
+<net name="E_A2" class="0">
+<segment>
+<pinref part="J9" gate="G$1" pin="5"/>
+<wire x1="55.88" y1="127" x2="43.18" y2="127" width="0.1524" layer="91"/>
+<label x="45.72" y="127" size="1.778" layer="95"/>
+</segment>
+</net>
+<net name="E_A1" class="0">
+<segment>
+<pinref part="J9" gate="G$1" pin="4"/>
+<wire x1="78.74" y1="124.46" x2="91.44" y2="124.46" width="0.1524" layer="91"/>
+<label x="83.82" y="124.46" size="1.778" layer="95"/>
+</segment>
+</net>
+<net name="E_B2" class="0">
+<segment>
+<pinref part="J9" gate="G$1" pin="6"/>
+<wire x1="78.74" y1="127" x2="91.44" y2="127" width="0.1524" layer="91"/>
+<label x="83.82" y="127" size="1.778" layer="95"/>
+</segment>
+</net>

Commit message: Add MPN for Q9
Parts:
- Q9: MPN (none) -> DMP3099L-13
Changed lines of the file:
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@@
 <attribute name="R" value="1k5"/>
 </part>
-<part name="Q9" library="robbe" deviceset="PFET" device="SM" package3d_urn="urn:adsk.eagle:package:2653225/3"/>
+<part name="Q9" library="robbe" deviceset="PFET" device="SM" package3d_urn="urn:adsk.eagle:package:2653225/3">
+<attribute name="MPN" value="DMP3099L-13"/>
+</part>
 <part name="+3V28" library="supply1" library_urn="urn:adsk.eagle:library:371" deviceset="+3V3" device=""/>
 <part name="C78" library="robbe" deviceset="C" device="">
@@
 <instance part="Q9" gate="G$1" x="185.42" y="144.78" smashed="yes">
 <attribute name="NAME" x="190.5" y="147.32" size="1.778" layer="95"/>
+<attribute name="MPN" x="185.42" y="144.78" size="1.778" layer="96" display="off"/>
 </instance>
 <instance part="+3V28" gate="G$1" x="185.42" y="154.94" smashed="yes">

Commit message: Move LED3 and LED4 on micro
Connections:
- net LED3: now also IC1.P0[17]/CTS1/MISO0/MISO; no longer IC1.P0[27]/SDA0/USB_SDA
- net LED4: now also IC1.P1[31]/SCK1/AD0[5]; no longer IC1.P0[28]/SCL0/USB_SCL
Changed lines of the file:
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@@
-</segment>
-</net>
-<net name="LED3" class="0">
-<segment>
-<pinref part="IC1" gate="G$1" pin="P0[27]/SDA0/USB_SDA"/>
-<wire x1="48.26" y1="177.8" x2="30.48" y2="177.8" width="0.1524" layer="91"/>
-<label x="30.48" y="177.8" size="1.778" layer="95"/>
-</segment>
-</net>
-<net name="LED4" class="0">
-<segment>
-<pinref part="IC1" gate="G$1" pin="P0[28]/SCL0/USB_SCL"/>
-<wire x1="48.26" y1="175.26" x2="30.48" y2="175.26" width="0.1524" layer="91"/>
-<label x="30.48" y="175.26" size="1.778" layer="95"/>
 </segment>
 </net>
@@
 </segment>
 </net>
+<net name="LED3" class="0">
+<segment>
+<pinref part="IC1" gate="G$1" pin="P0[17]/CTS1/MISO0/MISO"/>
+<wire x1="48.26" y1="203.2" x2="30.48" y2="203.2" width="0.1524" layer="91"/>
+<label x="30.48" y="203.2" size="1.778" layer="95"/>
+</segment>
+</net>
+<net name="LED4" class="0">
+<segment>
+<pinref part="IC1" gate="G$1" pin="P1[31]/SCK1/AD0[5]"/>
+<wire x1="137.16" y1="180.34" x2="160.02" y2="180.34" width="0.1524" layer="91"/>
+<label x="139.7" y="180.34" size="1.778" layer="95"/>
+</segment>
+</net>

Commit message: Swap PROBE and CONN
Connections:
- net SENSER_CONN: now also R51.1, R53.1; no longer R50.1, R52.1
- net SENSER_PROBE: now also R50.1, R52.1; no longer R51.1, R53.1
Changed lines of the file:
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@@
 <drawing>
 <settings>
-<setting alwaysvectorfont="no"/>
+<setting alwaysvectorfont="yes"/>
 <setting verticaltext="up"/>
 </settings>
@@
 </segment>
 </net>
-<net name="SENSER_CONN" class="0">
-<segment>
-<pinref part="R50" gate="G$1" pin="1"/>
-<wire x1="121.92" y1="60.96" x2="129.54" y2="60.96" width="0.1524" layer="91"/>
-<label x="142.24" y="60.96" size="1.778" layer="95"/>
-<pinref part="R52" gate="G$1" pin="1"/>
-<wire x1="129.54" y1="60.96" x2="160.02" y2="60.96" width="0.1524" layer="91"/>
-<wire x1="129.54" y1="63.5" x2="129.54" y2="60.96" width="0.1524" layer="91"/>
-<junction x="129.54" y="60.96"/>
-</segment>
-</net>
 <net name="N$63" class="0">
 <segment>
@@
 <net name="SENSER_PROBE" class="0">
 <segment>
+<pinref part="R50" gate="G$1" pin="1"/>
+<wire x1="121.92" y1="60.96" x2="129.54" y2="60.96" width="0.1524" layer="91"/>
+<pinref part="R52" gate="G$1" pin="1"/>
+<wire x1="129.54" y1="60.96" x2="160.02" y2="60.96" width="0.1524" layer="91"/>
+<wire x1="129.54" y1="63.5" x2="129.54" y2="60.96" width="0.1524" layer="91"/>
+<junction x="129.54" y="60.96"/>
+<label x="142.24" y="60.96" size="1.778" layer="95"/>
+</segment>
+</net>
+<net name="SENSER_CONN" class="0">
+<segment>
 <pinref part="R51" gate="G$1" pin="1"/>
 <wire x1="121.92" y1="55.88" x2="134.62" y2="55.88" width="0.1524" layer="91"/>
-<label x="142.24" y="55.88" size="1.778" layer="95"/>
 <pinref part="R53" gate="G$1" pin="1"/>
 <wire x1="134.62" y1="55.88" x2="160.02" y2="55.88" width="0.1524" layer="91"/>
 <wire x1="134.62" y1="63.5" x2="134.62" y2="55.88" width="0.1524" layer="91"/>
 <junction x="134.62" y="55.88"/>
+<label x="142.24" y="55.88" size="1.778" layer="95"/>
 </segment>
 </net>
