File: board/olchanowski.brd (EAGLE design)
At the start: 140 x 100 mm, 201 parts, among them IC1 LPC1768, J1 X-AXIS, J10 B4B-XH-A(LF)(SN), J2 Y-AXIS, J3 Z_AXIS, J4 ARJM11D7-009-AB-ER2-T, J5 RGB LED, J6 USB-C-FEMALE, J7 1744428-4, J8 282814-4, J9 1-281742-2, P1 TPSM53602, Q1 12MHz, Q10 SSM3K329R,LF, Q11 SSM3K329R,LF, Q2 25MHz, Q3 SIJA58DP, Q4 SIJA58DP, Q5 SSM3K329R,LF, Q6 SSM3K329R,LF, Q7 SSM3K329R,LF, Q8 SSM3K329R,LF, Q9 PFETSM, SW1 SPST-2-4PIN, SW2 SPST-2-4PIN, U1 TMC2209-LA, U2 TMC2209-LA, U3 TMC2209-LA, U4 TMC2209-LA, U5 LAN8720, U6 74HC1G04, U7 LM5111, U8 NCP5661-0, U9 PCA9306DCTR, X1 X-AXIS, X2 Y-AXIS, X3 Z-AXIS, X4 FAN, X5 LCD, X6 HB THERM, X7 SENSER

Commit message: Minor schematic improvements and initial routing work
Parts:
- C1, C10, C11, C12, C13, C14, C15, C17, C18, C19, C2, C20, C21, C22, C23, C24, C26, C27, C28, C29, C3, C30, C31, C32, C33, C35, C36, C37, C38, C39, C4, C40, C41, C42, C43, C44, C45, C46, C47, C48, C49, C5, C50, C51, C52, C53, C54, C55, C56, C57, C58, C59, C6, C60, C61, C62, C63, C64, C68, C72, C78, C79, C8, C80, C82, C83, C85, C86, C87, C88, C89, C9: value (none) -> C; device rcl:C0402 -> robbe:0402
- moved Q2 246.7 mm to (95.4, 90.1)
- moved R27 204.0 mm to (100.7, 88.7), turned to 180 degrees
- moved R26 197.1 mm to (98.9, 89.6), turned to 270 degrees
- moved R24 189.7 mm to (100.4, 77.9)
- moved R25 189.7 mm to (95.3, 77.9)
- moved R23 177.0 mm to (93.6, 86.0)
- moved R22 171.8 mm to (93.6, 87.0)
- moved R14 171.0 mm to (132.0, 75.7)
- moved R21 167.0 mm to (93.6, 85.0)
- moved R13 164.0 mm to (131.9, 93.7)
- moved R19 158.0 mm to (95.4, 92.2)
- moved R17 153.8 mm to (100.7, 85.5), turned to 180 degrees
- moved R16 148.5 mm to (100.7, 87.6), turned to 180 degrees
- moved C57 147.6 mm to (105.7, 95.5)
- moved C58 147.6 mm to (100.6, 95.5)
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
Commit message: Component placement
Parts:
- moved R44 266.8 mm to (154.0, 18.5)
- moved R45 266.8 mm to (148.9, 18.5)
- moved C78 253.1 mm to (146.7, 17.1)
- moved C79 251.2 mm to (145.2, 35.5)
- moved R49 246.3 mm to (116.7, 26.5), turned to 270 degrees
- moved Q11 244.6 mm to (119.1, 26.6)
- moved C82 244.3 mm to (129.9, 28.3), turned to 90 degrees
- moved R48 243.8 mm to (116.7, 32.1), turned to 270 degrees
- moved C83 242.9 mm to (129.7, 20.5), turned to 90 degrees
- moved Q10 242.8 mm to (119.7, 32.2)
- moved C32 236.7 mm to (119.1, 9.44)
- moved C81 236.2 mm to (120.9, 69.0), turned to 90 degrees
- moved J6 228.4 mm to (147.8, 25.4), turned to 90 degrees
- moved C84 227.3 mm to (117.4, 17.3)
- moved C31 220.1 mm to (109.2, 16.6)
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Connections:
- removed net ROT_B\: X5.12
- net ROT_B: now also X5.12
Other:
- board text added: "ICSP"
- board text added: "RESET"

Commit message: Example routing for a stepper driver
Parts:
- moved C83 81.0 mm to (58.6, 59.2), turned to 0 degrees
- moved C80 45.0 mm to (58.6, 60.3), turned to 180 degrees
- moved C42 31.2 mm to (45.5, 75.2)
- moved C40 23.3 mm to (52.4, 75.2)
- moved LED1 20.4 mm to (63.8, 93.7), turned to 0 degrees
- moved R28 18.7 mm to (20.7, 49.1)
- moved LED2 17.8 mm to (64.8, 93.7), turned to 0 degrees
- moved LED3 15.0 mm to (65.9, 93.7), turned to 0 degrees
- moved LED4 12.1 mm to (66.9, 93.7), turned to 0 degrees
- moved C43 12.0 mm to (57.9, 66.7), turned to 90 degrees
- moved R29 11.5 mm to (20.7, 48.0)
- moved C6 9.48 mm to (27.2, 15.7), turned to 180 degrees
- moved C8 7.20 mm to (18.3, 20.4), turned to 270 degrees
- moved R1 6.68 mm to (17.3, 14.2), turned to 180 degrees
- moved R30 6.47 mm to (20.7, 46.9)
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Routing:
- net N$11: track 0.00 -> 28.5 mm, vias 0 -> 5
- net +3V3: track 0.00 -> 19.7 mm
- net N$9: track 0.00 -> 17.4 mm, vias 0 -> 5
- net X_END: track 0.00 -> 16.9 mm
- net N$10: track 0.00 -> 12.6 mm, vias 0 -> 5
- net Y_END: track 0.00 -> 11.1 mm
- net N$8: track 0.00 -> 10.6 mm, vias 0 -> 5
- net ROT_A: track 0.00 -> 9.14 mm
- net +24V: track 0.00 -> 8.16 mm, vias 0 -> 13
- net TMC_ENN_X: track 0.00 -> 7.03 mm
- net BTN: track 0.00 -> 6.88 mm
- net N$2: track 0.00 -> 6.46 mm
- net N$38: track 0.00 -> 5.96 mm
- net N$45: track 0.00 -> 5.19 mm
- net Z_END: track 0.00 -> 4.99 mm
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- added copper zone on layer 1, net +24V
- added copper zone on layer 1, net N$10
- added copper zone on layer 16, net N$10
- added copper zone on layer 1, net N$11
- added copper zone on layer 16, net N$11
- added copper zone on layer 1, net N$8
- added copper zone on layer 16, net N$8
- added copper zone on layer 1, net N$9
- added copper zone on layer 16, net N$9

Commit message: More routing
Parts:
- removed C84: (no value), rcl:150CLZ-0810
- added C90, C91: C, robbe:0402
- moved C89 69.7 mm to (76.1, 90.5)
- moved R55 65.0 mm to (74.5, 86.5), turned to 180 degrees
- moved J10 65.0 mm to (83.0, 93.7)
- moved R54 62.3 mm to (74.5, 87.6), turned to 180 degrees
- moved Q9 62.0 mm to (90.1, 21.1)
- moved R44 61.9 mm to (92.1, 16.2), turned to 270 degrees
- moved C88 60.0 mm to (78.8, 93.2), turned to 90 degrees
- moved C87 60.0 mm to (76.3, 84.1)
- moved U9 58.5 mm to (77.4, 87.3), turned to 90 degrees
- moved J6 57.4 mm to (92.8, 8.88), turned to 0 degrees
- moved C79 56.4 mm to (91.6, 17.7), turned to 180 degrees
- moved R46 56.2 mm to (91.7, 18.8)
- moved R45 55.8 mm to (93.2, 16.2), turned to 270 degrees
- moved C78 53.0 mm to (93.7, 17.7)
- moved D2 51.3 mm to (96.1, 11.9), turned to 270 degrees
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Connections:
- net +24V: no longer C84.+
- net +3V3: now also C90.2, C91.2
- net +5V: no longer C70.1, C71.1, C72.2
- net BTN: now also IC1.85; no longer IC1.37
- net BUZZER_GATE: now also IC1.82; no longer IC1.38
- net GND: now also C90.1, C91.1; no longer C84.-
- net N$59: now also C70.1, C71.1, C72.2
Routing:
- net DP: track 0.00 -> 100.3 mm, vias 0 -> 2
- net DN: track 0.00 -> 100.1 mm
- net SD_MISO: track 0.00 -> 92.2 mm
- net SD_MOSI: track 0.00 -> 91.9 mm
- net BUZZER_GATE: track 0.00 -> 86.3 mm
- net SD_CLK: track 0.00 -> 82.7 mm
- net SD_CS: track 0.00 -> 78.8 mm
- net BTN: track 6.88 -> 82.6 mm
- net +24V: track 8.16 -> 74.2 mm, vias 13 -> 52
- net LCD_CS_N: track 0.00 -> 58.4 mm, vias 0 -> 2
- net LCD_SCLK: track 0.00 -> 56.5 mm, vias 0 -> 2
- net LCD_SDIN: track 0.00 -> 52.6 mm, vias 0 -> 2
- net +3V3: track 19.7 -> 61.0 mm
- net ENET_LED1: track 0.00 -> 39.4 mm, vias 0 -> 1
- net LCD_D/C_N: track 0.00 -> 36.3 mm
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- added copper zone on layer 16, net +24V
- added copper zone on layer 1, net +3V3
- added copper zone on layer 1, net +5V
- added copper zone on layer 1, net EXTR_HEATER
- added copper zone on layer 1, net E_A1
- added copper zone on layer 16, net E_A1
- added copper zone on layer 1, net E_A2
- added copper zone on layer 16, net E_A2
- added copper zone on layer 1, net E_B1
- added copper zone on layer 16, net E_B1
- added copper zone on layer 1, net E_B2
- added copper zone on layer 16, net E_B2
- added copper zone on layer 1, net N$18
- added copper zone on layer 16, net N$18
- added copper zone on layer 1, net N$19
- added copper zone on layer 16, net N$19
- added copper zone on layer 1, net N$20
- added copper zone on layer 16, net N$20
- added copper zone on layer 1, net N$21
- added copper zone on layer 16, net N$21
- added copper zone on layer 1, net N$28
- added copper zone on layer 16, net N$28
- added copper zone on layer 1, net N$29
- added copper zone on layer 16, net N$29
- added copper zone on layer 1, net N$30
- added copper zone on layer 16, net N$30
- added copper zone on layer 1, net N$31
- added copper zone on layer 16, net N$31
- added copper zone on layer 1, net N$59
- added copper zone on layer 1, net N$61
Other:
- board text added: "+3V3"
- board text added: "EXTR"
- board text added: "FILAMENT SENSOR"
- board text added: "HB"
- board text added: "USB"

Commit message: Routing
Parts:
- moved LED4 27.9 mm to (44.0, 77.8), turned to 270 degrees
- moved LED3 26.4 mm to (44.0, 78.9), turned to 270 degrees
- moved LED2 24.9 mm to (44.0, 79.9), turned to 270 degrees
- moved LED1 23.5 mm to (44.0, 81.0), turned to 270 degrees
- moved C80 1.91 mm to (47.0, 73.6)
- moved C83 1.91 mm to (48.1, 73.6)
- moved Q5 1.02 mm to (78.7, 39.0)
- moved R33 1.02 mm to (78.8, 36.6)
- moved X4 1.02 mm to (73.1, 39.1)
- moved C39 0.51 mm to (45.0, 73.1)
- moved L1 0.51 mm to (45.0, 74.1)
- moved C57 0.25 mm to (106.8, 90.2)
- moved C60 0.25 mm to (106.8, 89.1)
- moved U6 0.25 mm to (104.6, 81.0)
- moved C58 0.25 mm to (106.8, 88.1)
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Connections:
- net TMC_DIR_X: now also IC1.48; no longer IC1.80
- net TMC_DIR_Y: now also IC1.80; no longer IC1.49
- net TMC_ENN_X: now also IC1.49; no longer IC1.81
- net TMC_ENN_Y: now also IC1.81; no longer IC1.48
- net TMC_STEP_X: now also IC1.73; no longer IC1.75
- net TMC_STEP_Z: now also IC1.75; no longer IC1.73
Routing:
- net +3V3: track 61.0 -> 381.4 mm, vias 0 -> 14
- net +24V: track 74.2 -> 361.2 mm, vias 52 -> 106
- net TMC_STEP_E: track 0.00 -> 141.8 mm, vias 0 -> 4
- net TMC_DIR_E: track 0.00 -> 141.0 mm, vias 0 -> 4
- net HB_EN: track 10.3 -> 149.4 mm, vias 0 -> 4
- net EXTR_HEATER_EN: track 6.37 -> 143.8 mm, vias 0 -> 4
- net TMC_ENN_E: track 7.17 -> 142.1 mm, vias 0 -> 4
- net +5V: track 13.6 -> 148.1 mm, vias 0 -> 1
- net FAN1_EN: track 1.58 -> 132.3 mm, vias 0 -> 4
- net FAN2_EN: track 1.56 -> 128.6 mm, vias 0 -> 4
- net USB_CONNECT: track 0.00 -> 114.3 mm, vias 0 -> 4
- net FAN_EN: track 1.53 -> 105.0 mm, vias 0 -> 4
- net TMC_STEP_Z: track 0.00 -> 102.2 mm, vias 0 -> 4
- net TMC_ENN_Z: track 7.06 -> 108.5 mm, vias 0 -> 4
- net TMC_DIR_Z: track 0.00 -> 99.1 mm, vias 0 -> 4
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Other:
- board text added: "DEBUG"

Commit message: First rev done and ordered!
Parts:
- added R56: (no value), rcl:R0402
- moved R47 2.43 mm to (18.3, 38.9), turned to 180 degrees
- moved C17 0.57 mm to (42.8, 20.6)
- moved C26 0.38 mm to (68.1, 20.7)
- moved C8 0.36 mm to (18.0, 20.6)
- moved R22 0.13 mm to (97.8, 85.9)
- moved C80 0.13 mm to (47.1, 73.6)
- moved C55 0.13 mm to (97.8, 86.9)
- moved C56 0.13 mm to (97.8, 88.0)
- moved C59 0.13 mm to (97.8, 82.7)
- moved C61 0.13 mm to (97.8, 83.8)
- moved C83 0.13 mm to (48.2, 73.6)
- moved R23 0.13 mm to (97.8, 84.9)
- moved R31 0.13 mm to (109.7, 42.2)
- moved U6 0.13 mm to (104.6, 80.9)
Connections:
- removed net ENET_TXD_EN: IC1.93
- new net N$47: IC1.48, R56.1
- net ENET_TX_EN: now also IC1.93
- net TMC_DIR_X: now also IC1.38; no longer IC1.48
- net TMC_ENN_X: now also IC1.37; no longer IC1.49
- net TMC_UART: now also IC1.49, R56.2
Routing:
- net +3V3: track 381.4 -> 716.3 mm, vias 14 -> 27
- net EXTR_TEMP: track 3.07 -> 115.3 mm, vias 0 -> 3
- net TMC_UART: track 60.5 -> 158.2 mm, vias 3 -> 8
- net ENET_TX_EN: track 0.00 -> 64.9 mm, vias 0 -> 4
- net SCL: track 3.89 -> 62.4 mm, vias 0 -> 4
- net SDA: track 4.55 -> 62.7 mm, vias 0 -> 4
- net HB_TEMP: track 6.13 -> 58.0 mm, vias 0 -> 2
- net +24V: track 361.2 -> 398.4 mm, vias 106 -> 124
- net TMC_ENN_X: track 52.9 -> 59.9 mm, vias 0 -> 2
- net TMC_DIR_X: track 50.7 -> 57.3 mm, vias 0 -> 2
- net N$47: track 0.00 -> 4.92 mm
- net FAN1_EN: track 132.3 -> 133.6 mm
- net FAN2_EN: track 128.6 -> 129.5 mm
- net ENET_TXD1: track 65.5 -> 66.2 mm
- net ENET_TXD0: track 64.1 -> 64.7 mm
Other:
- board text added: "Olchanowski"
- board text added: "Robbe Derks - 2020"
- board text added: "v1.0"
