File: board/olchanowski.brd (EAGLE design)
At the start: 140 x 100 mm, 203 parts, among them IC1 LPC1768, J1 X-AXIS, J10 B4B-XH-A(LF)(SN), J2 Y-AXIS, J3 Z_AXIS, J4 ARJM11D7-009-AB-ER2-T, J5 RGB LED, J6 USB-C-FEMALE, J7 1744428-4, J8 282814-4, J9 1-281742-2, P1 TPSM53602, Q1 12MHz, Q10 SSM3K329R,LF, Q11 SSM3K329R,LF, Q2 25MHz, Q3 SIJA58DP, Q4 SIJA58DP, Q5 SSM3K329R,LF, Q6 SSM3K329R,LF, Q7 SSM3K329R,LF, Q8 SSM3K329R,LF, Q9 PFETSM, SW1 SPST-2-4PIN, SW2 SPST-2-4PIN, U1 TMC2209-LA, U2 TMC2209-LA, U3 TMC2209-LA, U4 TMC2209-LA, U5 LAN8720, U6 74HC1G04, U7 LM5111, U8 NCP5661-0, U9 PCA9306DCTR, X1 X-AXIS, X2 Y-AXIS, X3 Z-AXIS, X4 FAN, X5 LCD, X6 HB THERM, X7 SENSER

Commit message: Fix P1 NC/AGND pins
Connections:
- net GND: now also P1.10, P1.11, P1.12, P1.3

Commit message: Fix Stepper connector pinout
Connections:
- removed net N$28: J3.1, U3.24
- removed net N$30: J3.3, U3.21
- removed net N$31: J3.4, U3.1
- new net N$66: J1.4, U1.21
- new net N$68: J1.3, U1.24
- new net N$70: J1.1, U1.1
- net E_A1: now also J9.4; no longer J9.3
- net E_B1: now also J9.3; no longer J9.4
- net N$10: now also J2.3, U2.24; no longer J1.3, U1.21
- net N$11: now also J2.4, U2.21; no longer J1.4, U1.1
- net N$18: now also J3.1, U3.1; no longer J2.1, U2.24
- net N$20: now also J3.3, U3.24; no longer J2.3, U2.21
- net N$21: now also J3.4, U3.21; no longer J2.4, U2.1
- net N$8: now also J2.1, U2.1; no longer J1.1, U1.24
Routing:
- net N$31: track 28.6 -> 0.00 mm, vias 5 -> 0
- net N$21: track 28.6 -> 11.7 mm
- net N$11: track 28.5 -> 11.7 mm
- net E_B1: track 7.89 -> 22.3 mm
- net N$30: track 12.6 -> 0.00 mm, vias 5 -> 0
- net N$70: track 0.00 -> 11.8 mm, vias 0 -> 5
- net N$66: track 0.00 -> 11.7 mm, vias 0 -> 5
- net E_A1: track 17.4 -> 6.54 mm
- net N$28: track 10.7 -> 0.00 mm, vias 5 -> 0
- net N$68: track 0.00 -> 9.41 mm, vias 0 -> 5
- net N$19: track 17.4 -> 9.17 mm
- net N$9: track 17.4 -> 9.15 mm
- net N$69: track 17.4 -> 9.19 mm
- net N$20: track 12.6 -> 9.43 mm
- net N$10: track 12.6 -> 9.42 mm
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- added copper zone on layer 1, net N$66
- added copper zone on layer 16, net N$66
- added copper zone on layer 1, net N$68
- added copper zone on layer 16, net N$68
- added copper zone on layer 1, net N$70
- added copper zone on layer 16, net N$70
- removed copper zone on layer 1, net N$28
- removed copper zone on layer 16, net N$28
- removed copper zone on layer 1, net N$30
- removed copper zone on layer 16, net N$30
- removed copper zone on layer 1, net N$31
- removed copper zone on layer 16, net N$31

Commit message: Fix Ethernet pinout and LED position
Parts:
- moved C49 3.17 mm to (112.8, 83.1)
- moved R15 3.17 mm to (115.2, 83.1)
- moved R18 3.07 mm to (115.2, 86.1)
- moved C52 3.07 mm to (112.8, 86.2)
- moved C50 1.09 mm to (112.8, 84.1)
- moved R16 1.09 mm to (115.2, 84.1)
- moved R17 0.99 mm to (115.2, 85.1)
- moved C51 0.99 mm to (112.8, 85.1)
- moved R27 0.64 mm to (106.1, 86.8)
Routing:
- net N$43: track 17.2 -> 20.6 mm
- net N$40: track 18.6 -> 21.7 mm
- net N$39: track 21.5 -> 19.0 mm
- net N$41: track 20.8 -> 18.7 mm
- net N$45: track 5.19 -> 3.10 mm
- net N$54: track 1.46 -> 0.83 mm
- net ENET_LED1: track 39.4 -> 38.9 mm

Commit message: Move LED3 and LED4 on micro
Connections:
- net LED3: now also IC1.61; no longer IC1.25
- net LED4: now also IC1.20; no longer IC1.24
Routing:
- net LED3: track 17.0 -> 26.2 mm, vias 0 -> 2
- net LED4: track 16.2 -> 8.39 mm
Changed lines of the file:
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@@
 <wire x1="36.22" y1="68.153" x2="34.1" y2="68.153" width="0.254" layer="1"/>
 <wire x1="34.1" y1="68.153" x2="33.97" y2="68.023" width="0.254" layer="1"/>
-<wire x1="42" y1="73.013" x2="40.97" y2="71.983" width="0.254" layer="1"/>
-<wire x1="40.97" y1="71.983" x2="40.97" y2="70.903" width="0.254" layer="1"/>
+<wire x1="42" y1="73.013" x2="42" y2="72.72851875" width="0.254" layer="1"/>
+<wire x1="42" y1="72.72851875" x2="40.97" y2="71.69851875" width="0.254" layer="1"/>
+<wire x1="40.97" y1="71.69851875" x2="40.97" y2="70.903" width="0.254" layer="1"/>
 <wire x1="53.92" y1="61.026" x2="53.793" y2="61.153" width="0.254" layer="1"/>
 <wire x1="53.793" y1="61.153" x2="51.72" y2="61.153" width="0.254" layer="1"/>
@@
 <wire x1="37.658" y1="61.153" x2="36.22" y2="61.153" width="0.254" layer="1"/>
 <wire x1="39.47" y1="55.403" x2="39.47" y2="57.14218125" width="0.3048" layer="1"/>
-<wire x1="41.038" y1="58.71018125" x2="41.038" y2="63.12515625" width="0.3048" layer="1"/>
+<wire x1="40.954178125" y1="58.626359375" x2="40.954178125" y2="63.12515625" width="0.3048" layer="1"/>
 <via x="41.2666" y="63.35375625" extent="1-16" drill="0.35"/>
-<wire x1="39.47" y1="57.14218125" x2="41.038" y2="58.71018125" width="0.3048" layer="1"/>
+<wire x1="39.47" y1="57.14218125" x2="40.954178125" y2="58.626359375" width="0.3048" layer="1"/>
 <wire x1="36.22" y1="68.153" x2="37.165" y2="68.153" width="0.254" layer="1"/>
 <wire x1="37.165" y1="68.153" x2="37.211" y2="68.199" width="0.254" layer="1"/>
@@
 <wire x1="39.8611" y1="64.62375625" x2="39.8611" y2="68.199" width="0.254" layer="1"/>
 <wire x1="45.4798" y1="75.0894" x2="45.4474" y2="75.057" width="0.254" layer="16"/>
-<wire x1="45.4474" y1="75.057" x2="43.688" y2="75.057" width="0.254" layer="16"/>
-<wire x1="43.688" y1="75.057" x2="42.9006" y2="74.2696" width="0.254" layer="16"/>
-<wire x1="42.9006" y1="69.98784375" x2="43.0785" y2="69.80994375" width="0.254" layer="16"/>
-<wire x1="43.0785" y1="69.80994375" x2="43.0785" y2="65.17884375" width="0.254" layer="16"/>
-<wire x1="43.0785" y1="65.17884375" x2="41.2534125" y2="63.35375625" width="0.254" layer="16"/>
-<wire x1="42.9006" y1="74.2696" x2="42.9006" y2="69.98784375" width="0.254" layer="16"/>
+<wire x1="45.4474" y1="75.057" x2="44.0055" y2="75.057" width="0.254" layer="16"/>
+<wire x1="44.0055" y1="75.057" x2="43.416321875" y2="74.467821875" width="0.254" layer="16"/>
+<wire x1="43.416321875" y1="65.516665625" x2="41.2534125" y2="63.35375625" width="0.254" layer="16"/>
+<wire x1="43.416321875" y1="74.467821875" x2="43.416321875" y2="65.516665625" width="0.254" layer="16"/>
 <wire x1="128.1176" y1="30.51580625" x2="126.58" y2="28.97820625" width="0.508" layer="16"/>
 <wire x1="126.58" y1="28.91" x2="126.58" y2="28.97820625" width="0.508" layer="16"/>
@@
 <wire x1="68.0788" y1="20.169" x2="68.0788" y2="19.9898" width="0.3048" layer="1"/>
 <wire x1="68.5686" y1="19.5" x2="68.0788" y2="19.9898" width="0.3048" layer="1"/>
-<wire x1="41.038" y1="63.12515625" x2="41.2666" y2="63.35375625" width="0.3048" layer="1"/>
+<wire x1="41.182778125" y1="63.35375625" x2="41.2666" y2="63.35375625" width="0.3048" layer="1"/>
+<wire x1="41.182778125" y1="63.35375625" x2="40.954178125" y2="63.12515625" width="0.3048" layer="1"/>
 <wire x1="41.2666" y1="63.35375625" x2="41.1311" y2="63.35375625" width="0.3048" layer="16"/>
 <wire x1="41.1311" y1="63.35375625" x2="41.066428125" y2="63.418428125" width="0.3048" layer="16"/>
@@
 <wire x1="38.97" y1="53.173" x2="38.91" y2="53.113" width="0.127" layer="1"/>
 <via x="42.562" y="69.596" extent="1-16" drill="0.35"/>
-<wire x1="42.562" y1="69.596" x2="40.6485" y2="67.6825" width="0.2032" layer="1"/>
-<wire x1="40.6485" y1="58.8595" x2="39.0716" y2="57.2826" width="0.2032" layer="1"/>
+<wire x1="42.562" y1="69.596" x2="40.554521875" y2="67.588521875" width="0.2032" layer="1"/>
+<wire x1="40.554521875" y1="58.765521875" x2="39.0716" y2="57.2826" width="0.2032" layer="1"/>
 <wire x1="39.0716" y1="57.2826" x2="39.0716" y2="56.2666" width="0.2032" layer="1"/>
 <wire x1="39.0716" y1="56.2666" x2="38.97" y2="56.165" width="0.2032" layer="1"/>
 <wire x1="38.97" y1="55.403" x2="38.97" y2="56.165" width="0.2032" layer="1"/>
-<wire x1="40.6485" y1="67.6825" x2="40.6485" y2="58.8595" width="0.2032" layer="1"/>
+<wire x1="40.554521875" y1="67.588521875" x2="40.554521875" y2="58.765521875" width="0.2032" layer="1"/>
 <wire x1="42.562" y1="69.596" x2="42.545" y2="69.613" width="0.2032" layer="16"/>
 <wire x1="42.545" y1="75.014925" x2="42.121925" y2="75.438" width="0.2032" layer="16"/>
@@
 <wire x1="31.3394625" y1="60.8219625" x2="31.9686" y2="61.4511" width="0.2032" layer="16"/>
 <wire x1="31.9686" y1="61.4511" x2="32.8637875" y2="61.4511" width="0.2032" layer="16"/>
-<via x="41.656" y="60.071" extent="1-16" drill="0.35"/>
-<wire x1="41.656" y1="60.071" x2="45.97" y2="64.385" width="0.2032" layer="1"/>
-<wire x1="45.97" y1="64.385" x2="45.97" y2="70.903" width="0.2032" layer="1"/>
+<via x="41.887140625" y="60.071" extent="1-16" drill="0.35"/>
+<wire x1="41.887140625" y1="60.071" x2="45.97" y2="64.153859375" width="0.2032" layer="1"/>
+<wire x1="45.97" y1="64.153859375" x2="45.97" y2="70.903" width="0.2032" layer="1"/>
 <wire x1="20.4216" y1="40.5376" x2="20.4216" y2="44.485175" width="0.2032" layer="1"/>
 <wire x1="20.4216" y1="44.485175" x2="30.4546" y2="54.518175" width="0.2032" layer="1"/>
 <wire x1="30.4546" y1="54.518175" x2="30.4546" y2="57.479875" width="0.2032" layer="1"/>
 <wire x1="30.3106" y1="59.56555" x2="31.3394625" y2="60.5944125" width="0.2032" layer="16"/>
-<wire x1="34.2438875" y1="60.071" x2="41.656" y2="60.071" width="0.2032" layer="16"/>
+<wire x1="34.2438875" y1="60.071" x2="41.887140625" y2="60.071" width="0.2032" layer="16"/>
 </signal>
 <signal name="N$3">
@@
 </signal>
 <signal name="LED3">
-<contactref element="IC1" pad="25"/>
 <contactref element="LED3" pad="A"/>
-<wire x1="43.2652" y1="78.8904" x2="43.1823125" y2="78.8904" width="0.2032" layer="1"/>
-<wire x1="43.1823125" y1="78.8904" x2="42.4619125" y2="78.17" width="0.2032" layer="1"/>
-<wire x1="34.8488" y1="75.447775" x2="34.8488" y2="72.634225" width="0.2032" layer="1"/>
-<wire x1="35.550225" y1="71.9328" x2="37.8206" y2="71.9328" width="0.2032" layer="1"/>
-<wire x1="37.571025" y1="78.17" x2="34.8488" y2="75.447775" width="0.2032" layer="1"/>
-<wire x1="34.8488" y1="72.634225" x2="35.550225" y2="71.9328" width="0.2032" layer="1"/>
-<wire x1="37.8206" y1="71.9328" x2="37.97" y2="71.7834" width="0.2032" layer="1"/>
-<wire x1="37.97" y1="71.7834" x2="37.97" y2="70.903" width="0.2032" layer="1"/>
-<wire x1="42.4619125" y1="78.17" x2="37.571025" y2="78.17" width="0.2032" layer="1"/>
+<contactref element="IC1" pad="61"/>
+<wire x1="43.2652" y1="78.8904" x2="42.540459375" y2="78.8904" width="0.2032" layer="1"/>
+<wire x1="42.540459375" y1="78.8904" x2="42.52721875" y2="78.877159375" width="0.2032" layer="1"/>
+<via x="42.52721875" y="78.877159375" extent="1-16" drill="0.35"/>
+<wire x1="42.52721875" y1="78.877159375" x2="42.52721875" y2="75.49968125" width="0.2032" layer="16"/>
+<wire x1="42.52721875" y1="75.49968125" x2="43.060725" y2="74.966175" width="0.2032" layer="16"/>
+<wire x1="43.060725" y1="65.92658125" x2="42.899825" y2="65.76568125" width="0.2032" layer="16"/>
+<via x="42.899825" y="65.76568125" extent="1-16" drill="0.35"/>
+<wire x1="42.899825" y1="65.76568125" x2="42.899825" y2="63.02535" width="0.2032" layer="1"/>
+<wire x1="42.899825" y1="63.02535" x2="41.3453375" y2="61.4708625" width="0.2032" layer="1"/>
+<wire x1="43.060725" y1="74.966175" x2="43.060725" y2="65.92658125" width="0.2032" layer="16"/>
+<wire x1="41.9887375" y1="59.18708125" x2="42.687240625" y2="59.18708125" width="0.2032" layer="1"/>
+<wire x1="42.687240625" y1="59.18708125" x2="42.97" y2="58.904321875" width="0.2032" layer="1"/>
+<wire x1="42.97" y1="58.904321875" x2="42.97" y2="55.403" width="0.2032" layer="1"/>
+<wire x1="41.3453375" y1="61.4708625" x2="41.3453375" y2="59.83048125" width="0.2032" layer="1"/>
+<wire x1="41.3453375" y1="59.83048125" x2="41.9887375" y2="59.18708125" width="0.2032" layer="1"/>
 </signal>
 <signal name="LED4">
-<contactref element="IC1" pad="24"/>
 <contactref element="LED4" pad="A"/>
-<wire x1="38.47" y1="70.903" x2="38.47" y2="71.766" width="0.2032" layer="1"/>
-<wire x1="35.687" y1="72.263" x2="35.179" y2="72.771" width="0.2032" layer="1"/>
-<wire x1="35.179" y1="72.771" x2="35.179" y2="75.311" width="0.2032" layer="1"/>
-<wire x1="37.7078" y1="77.8398" x2="43.255" y2="77.8398" width="0.2032" layer="1"/>
-<wire x1="38.47" y1="71.766" x2="37.973" y2="72.263" width="0.2032" layer="1"/>
-<wire x1="37.973" y1="72.263" x2="35.687" y2="72.263" width="0.2032" layer="1"/>
-<wire x1="35.179" y1="75.311" x2="37.7078" y2="77.8398" width="0.2032" layer="1"/>
+<contactref element="IC1" pad="20"/>
+<wire x1="43.255" y1="77.8398" x2="42.736840625" y2="77.8398" width="0.2032" layer="1"/>
+<wire x1="42.736840625" y1="77.8398" x2="41.450259375" y2="76.55321875" width="0.2032" layer="1"/>
+<wire x1="40.47" y1="71.70141875" x2="40.47" y2="70.903" width="0.2032" layer="1"/>
+<wire x1="41.450259375" y1="76.55321875" x2="41.450259375" y2="72.681678125" width="0.2032" layer="1"/>
+<wire x1="41.450259375" y1="72.681678125" x2="40.47" y2="71.70141875" width="0.2032" layer="1"/>
 </signal>
 <signal name="N$67">

Commit message: Drill hole for JST plus some clean ups
Routing:
- net X_END: track 56.4 -> 57.3 mm
- net +3V3: track 716.3 -> 717.1 mm
- net SENSER_CONN: track 62.3 -> 63.0 mm
- net SENSER_PROBE: track 70.2 -> 70.8 mm

Commit message: Swap PROBE and CONN
Connections:
- net SENSER_CONN: now also R51.1, R53.1; no longer R50.1, R52.1
- net SENSER_PROBE: now also R50.1, R52.1; no longer R51.1, R53.1
Routing:
- net SENSER_PROBE: track 70.8 -> 63.0 mm
- net SENSER_CONN: track 63.0 -> 70.7 mm
Changed lines of the file:
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@@
 <drawing>
 <settings>
-<setting alwaysvectorfont="no"/>
+<setting alwaysvectorfont="yes"/>
 <setting verticaltext="up"/>
 </settings>
@@
 <signal name="SENSER_PROBE">
 <contactref element="IC1" pad="26"/>
-<contactref element="R51" pad="1"/>
-<contactref element="R53" pad="1"/>
-<wire x1="8.9418" y1="29.5754" x2="10.032" y2="29.5754" width="0.127" layer="1"/>
-<wire x1="10.032" y1="29.5754" x2="10.0508" y2="29.5942" width="0.127" layer="1"/>
-<wire x1="10.0508" y1="29.5942" x2="10.668" y2="30.2114" width="0.2032" layer="1"/>
-<wire x1="10.4344875" y1="37.3808" x2="9.928175" y2="37.3808" width="0.2032" layer="1"/>
-<wire x1="10.668" y1="30.2114" x2="10.668" y2="37.1472875" width="0.2032" layer="1"/>
-<wire x1="10.668" y1="37.1472875" x2="10.4344875" y2="37.3808" width="0.2032" layer="1"/>
-<wire x1="10.1855" y1="62.2926" x2="10.1855" y2="62.441475" width="0.2032" layer="1"/>
-<via x="10.1855" y="62.441475" extent="1-16" drill="0.35"/>
-<wire x1="10.1855" y1="62.441475" x2="10.1855" y2="62.669025" width="0.2032" layer="16"/>
+<wire x1="1.285240625" y1="46.062896875" x2="1.285234375" y2="53.3938875" width="0.2032" layer="1"/>
+<wire x1="9.741" y1="61.849653125" x2="1.285234375" y2="53.3938875" width="0.2032" layer="1"/>
+<wire x1="9.741" y1="61.849653125" x2="9.741" y2="62.113815625" width="0.2032" layer="1"/>
+<via x="9.741" y="62.113815625" extent="1-16" drill="0.35"/>
+<wire x1="9.741" y1="62.113815625" x2="9.7537" y2="62.113815625" width="0.2032" layer="16"/>
+<wire x1="15.979184375" y1="68.3393" x2="9.7537" y2="62.113815625" width="0.2032" layer="16"/>
 <wire x1="32.9861" y1="68.3393" x2="33.147" y2="68.1784" width="0.2032" layer="16"/>
 <via x="33.147" y="68.1784" extent="1-16" drill="0.35"/>
@@
 <wire x1="36.2124" y1="69.1606" x2="36.22" y2="69.153" width="0.2032" layer="1"/>
 <wire x1="33.147" y1="68.1784" x2="34.1292" y2="69.1606" width="0.2032" layer="1"/>
-<wire x1="9.928175" y1="37.3808" x2="1.6865625" y2="45.6224125" width="0.2032" layer="1"/>
-<wire x1="1.6865625" y1="45.6224125" x2="1.6865625" y2="53.7936625" width="0.2032" layer="1"/>
-<wire x1="1.6865625" y1="53.7936625" x2="10.1855" y2="62.2926" width="0.2032" layer="1"/>
-<wire x1="10.1855" y1="62.669025" x2="15.855775" y2="68.3393" width="0.2032" layer="16"/>
-<wire x1="15.855775" y1="68.3393" x2="32.9861" y2="68.3393" width="0.2032" layer="16"/>
-</signal>
-<signal name="SENSER_CONN">
-<contactref element="IC1" pad="27"/>
+<wire x1="15.979184375" y1="68.3393" x2="32.9861" y2="68.3393" width="0.2032" layer="16"/>
 <contactref element="R50" pad="1"/>
 <contactref element="R52" pad="1"/>
 <wire x1="8.889" y1="36.8456" x2="9.9832" y2="36.8456" width="0.127" layer="1"/>
 <wire x1="9.9832" y1="36.8456" x2="9.9898" y2="36.8522" width="0.127" layer="1"/>
-<wire x1="9.9898" y1="36.8522" x2="1.35128125" y2="45.49071875" width="0.2032" layer="1"/>
-<wire x1="9.5335" y1="62.107575" x2="9.5335" y2="62.484" width="0.2032" layer="1"/>
-<via x="9.5335" y="62.484" extent="1-16" drill="0.35"/>
-<wire x1="9.5335" y1="62.484" x2="15.719" y2="68.6695" width="0.2032" layer="16"/>
-<wire x1="15.719" y1="68.6695" x2="34.925" y2="68.6695" width="0.2032" layer="16"/>
+<wire x1="9.9898" y1="36.8522" x2="9.9898" y2="37.3583375" width="0.2032" layer="1"/>
+<wire x1="9.9898" y1="37.3583375" x2="1.285240625" y2="46.062896875" width="0.2032" layer="1"/>
+</signal>
+<signal name="SENSER_CONN">
+<contactref element="IC1" pad="27"/>
+<via x="10.112621875" y="63.1698" extent="1-16" drill="0.35"/>
+<wire x1="10.112621875" y1="63.1698" x2="15.612321875" y2="68.6695" width="0.2032" layer="16"/>
+<wire x1="15.612321875" y1="68.6695" x2="34.925" y2="68.6695" width="0.2032" layer="16"/>
 <via x="34.925" y="68.6695" extent="1-16" drill="0.35"/>
 <wire x1="34.925" y1="68.6695" x2="34.9415" y2="68.653" width="0.2032" layer="1"/>
 <wire x1="34.9415" y1="68.653" x2="36.22" y2="68.653" width="0.2032" layer="1"/>
-<wire x1="1.35128125" y1="45.49071875" x2="1.35128125" y2="53.92535625" width="0.2032" layer="1"/>
-<wire x1="1.35128125" y1="53.92535625" x2="9.5335" y2="62.107575" width="0.2032" layer="1"/>
+<contactref element="R51" pad="1"/>
+<contactref element="R53" pad="1"/>
+<wire x1="8.9418" y1="29.5754" x2="10.032" y2="29.5754" width="0.127" layer="1"/>
+<wire x1="10.032" y1="29.5754" x2="10.0508" y2="29.5942" width="0.127" layer="1"/>
+<wire x1="10.112621875" y1="63.1698" x2="10.2321" y2="63.050321875" width="0.2032" layer="1"/>
+<wire x1="10.2321" y1="63.050321875" x2="10.2321" y2="61.8703" width="0.2032" layer="1"/>
+<wire x1="10.2321" y1="61.8703" x2="1.623065625" y2="53.261265625" width="0.2032" layer="1"/>
+<wire x1="10.68831875" y1="30.23171875" x2="10.0508" y2="29.5942" width="0.2032" layer="1"/>
+<wire x1="1.623065625" y1="53.261265625" x2="1.623065625" y2="46.19221875" width="0.2032" layer="1"/>
+<wire x1="10.68831875" y1="37.126965625" x2="10.68831875" y2="30.23171875" width="0.2032" layer="1"/>
+<wire x1="1.623065625" y1="46.19221875" x2="10.68831875" y2="37.126965625" width="0.2032" layer="1"/>
 </signal>
 <signal name="N$62">
